File: bench_stm32_esc/bench_stm32_esc.kicad_pcb (KiCad board)
At the start: 4 copper layers, 80 x 80 mm, 85 parts, among them J1 USB_C_Receptacle_USB2.0_16P, J2 XT60PW-M, Q1 CSD19532Q5B, Q2 CSD19532Q5B, U1 UCC27211ADRMR, U10 AS5047D, U11 USBLC6-2P6, U12 MR60PW-M.G.B, U4 AP2112K-3.3, U5 INA240A2D, U6 STM32G474RETx, U8 LM5164DDA, U9 TPD1E05U06DYA, X1 X322516MLB4SI

Commit message: Almost done rev 1.1
Parts:
- removed L2: SM7850-680MT, footprints:SM7850-680MT
- removed Q1, Q2: CSD19532Q5B, Package_TO_SOT_SMD:TDSON-8-1
- removed TP1: TestPoint, TestPoint:TestPoint_Pad_1.5x1.5mm
- removed U9: TPD1E05U06DYA, PCM_JLCPCB:D_SOD-523
- added C100: 100nF, PCM_JLCPCB:C_0402, B.Cu at (174.1, 70.0)
- added C101: 1nF, PCM_JLCPCB:C_0402, F.Cu at (47.3, 46.2)
- added C102: 1nF, PCM_JLCPCB:C_0402, F.Cu at (47.3, 48.1)
- added C103: 1nF, PCM_JLCPCB:C_0402, F.Cu at (47.3, 50.0)
- added C104: 1nF, PCM_JLCPCB:C_0402, F.Cu at (47.3, 51.8)
- added C105: FS55X226K101LRG, easyeda2kicad:C2220, F.Cu at (184.5, 116.4)
- added C106: FS55X226K101LRG, easyeda2kicad:C2220, F.Cu at (190.8, 116.4)
- added C107: 100nF, PCM_JLCPCB:C_0402, F.Cu at (159.4, 98.8)
- added C108: 1nF, PCM_JLCPCB:C_0402, F.Cu at (164.4, 66.0)
- added C109: 1nF, PCM_JLCPCB:C_0402, F.Cu at (161.3, 62.3)
- added C110: 1nF, PCM_JLCPCB:C_0402, F.Cu at (160.4, 81.8)
- added C111: 1nF, PCM_JLCPCB:C_0402, F.Cu at (164.5, 85.1)
- added C112: 1nF, PCM_JLCPCB:C_0402, F.Cu at (160.5, 98.0)
- added C113: 1nF, PCM_JLCPCB:C_0402, F.Cu at (164.7, 101.6)
- added C114: 1nF, PCM_JLCPCB:C_0402, F.Cu at (78.4, 55.7)
- added C24: 1uF, PCM_JLCPCB:C_0805, F.Cu at (180.5, 71.3)
- added C30: 47pF, PCM_JLCPCB:C_0402, B.Cu at (171.5, 67.3)
- added C33: 47pF, PCM_JLCPCB:C_0402, B.Cu at (170.3, 102.2)
- added C35: 100nF, PCM_JLCPCB:C_0402, B.Cu at (170.6, 84.6)
- added C38: 100nF, PCM_JLCPCB:C_0402, F.Cu at (171.1, 62.1)
- added C40: 100nF, PCM_JLCPCB:C_0402, F.Cu at (169.7, 61.7)
- added C43: 220nF, PCM_JLCPCB:C_0805, B.Cu at (177.9, 89.7)
- added C47: 1uF, PCM_JLCPCB:C_0805, F.Cu at (175.7, 89.7)
- added C48: 1uF, PCM_JLCPCB:C_0805, F.Cu at (177.9, 89.8)
- added C49: 1uF, PCM_JLCPCB:C_0805, F.Cu at (180.0, 89.8)
- added C50: 100nF, PCM_JLCPCB:C_0402, B.Cu at (170.3, 101.0)
- added C51: 1nF, PCM_JLCPCB:C_0402, F.Cu at (157.3, 57.9)
- added C52: 100nF, PCM_JLCPCB:C_0402, B.Cu at (172.3, 106.3)
- added C53: 100nF, PCM_JLCPCB:C_0402, B.Cu at (172.7, 104.9)
- added C54: 100nF, PCM_JLCPCB:C_0402, F.Cu at (160.2, 63.2)
- added C55: 10uF, PCM_JLCPCB:C_0402, B.Cu at (170.6, 83.5)
- added C56: 220nF, PCM_JLCPCB:C_0805, B.Cu at (180.5, 71.3)
- added C57: 220nF, PCM_JLCPCB:C_0805, B.Cu at (178.4, 71.3)
- added C58: 220nF, PCM_JLCPCB:C_0805, B.Cu at (176.3, 71.3)
- added C59: 1uF, PCM_JLCPCB:C_0805, F.Cu at (175.2, 106.2)
- added C60: 1uF, PCM_JLCPCB:C_0805, F.Cu at (177.3, 106.2)
- added C61: 1uF, PCM_JLCPCB:C_0805, F.Cu at (179.4, 106.2)
- added C62: 100nF, PCM_JLCPCB:C_0402, F.Cu at (44.5, 42.5)
- added C63: 100nF, PCM_JLCPCB:C_0402, F.Cu at (44.5, 44.4)
- added C64: 33nF, PCM_JLCPCB:C_0603, F.Cu at (172.6, 54.4)
- added C65: 33nF, PCM_JLCPCB:C_0603, F.Cu at (48.3, 65.1)
- added C66: 1nF, PCM_JLCPCB:C_0402, F.Cu at (157.1, 76.3)
- added C67: 1nF, PCM_JLCPCB:C_0402, F.Cu at (158.5, 92.3)
- added C68: 1.5nF, PCM_JLCPCB:C_0603, F.Cu at (171.6, 77.8)
- added C69: 1nF, PCM_JLCPCB:C_0402, F.Cu at (157.3, 61.2)
- added C70: 1nF, PCM_JLCPCB:C_0402, F.Cu at (157.2, 80.3)
- added C71: 33nF, PCM_JLCPCB:C_0603, F.Cu at (171.0, 73.1)
- added C72: 1.5nF, PCM_JLCPCB:C_0603, F.Cu at (170.8, 94.0)
- added C73: 1nF, PCM_JLCPCB:C_0402, F.Cu at (158.5, 96.0)
- added C74: 10uF, PCM_JLCPCB:C_0402, B.Cu at (171.5, 65.1)
- added C75: 33nF, PCM_JLCPCB:C_0603, F.Cu at (170.1, 89.2)
- added C76: 100nF, PCM_JLCPCB:C_0402, F.Cu at (47.3, 31.4)
- added C77: FS55X226K101LRG, easyeda2kicad:C2220, B.Cu at (184.5, 116.4)
- added C78: FS55X226K101LRG, easyeda2kicad:C2220, B.Cu at (178.2, 116.4)
- added C79: FS55X226K101LRG, easyeda2kicad:C2220, F.Cu at (178.2, 116.4)
- added C80: FS55X226K101LRG, easyeda2kicad:C2220, B.Cu at (190.8, 116.4)
- added C82: FS55X226K101LRG, easyeda2kicad:C2220, F.Cu at (169.9, 119.1)
- added C83: 100nF, PCM_JLCPCB:C_0402, F.Cu at (134.9, 100.8)
- added C84: 1.5nF, PCM_JLCPCB:C_0603, F.Cu at (70.9, 62.4)
- added C85: 18pF, PCM_JLCPCB:C_0402, F.Cu at (47.3, 33.3)
- added C86: 100nF, PCM_JLCPCB:C_0402, F.Cu at (159.4, 82.4)
- added C87: 18pF, PCM_JLCPCB:C_0402, F.Cu at (47.3, 35.1)
- added C88: 100nF, PCM_JLCPCB:C_0603, F.Cu at (155.3, 119.8)
- added C89: 18pF, PCM_JLCPCB:C_0603, F.Cu at (149.1, 116.1)
- added C90: 15uF, PCM_JLCPCB:C_0603, F.Cu at (140.2, 116.5)
- added C91: 15uF, PCM_JLCPCB:C_0603, F.Cu at (140.2, 115.2)
- added C92: 100nF, PCM_JLCPCB:C_0603, F.Cu at (151.9, 108.6)
- added C93: 1uF, PCM_JLCPCB:C_0402, F.Cu at (47.3, 37.0)
- added C94: 4.7uF, PCM_JLCPCB:C_1206, F.Cu at (151.9, 106.7)
- added C95: 1.5nF, PCM_JLCPCB:C_0603, F.Cu at (173.0, 59.1)
- added C96: 10uF, PCM_JLCPCB:C_0402, B.Cu at (170.3, 100.1)
- added C97: 100nF, PCM_JLCPCB:C_0402, B.Cu at (172.7, 89.9)
- added C98: 100nF, PCM_JLCPCB:C_0402, B.Cu at (173.2, 88.5)
- added C99: 100nF, PCM_JLCPCB:C_0402, B.Cu at (173.6, 71.4)
- added D4: Red, PCM_JLCPCB:D_0805, F.Cu at (26.1, 71.4)
- added D5: White, PCM_JLCPCB:D_0805, F.Cu at (26.1, 74.5)
- added FB4: ~, PCM_JLCPCB:R_0402, F.Cu at (168.3, 81.3)
- added FB5: ~, PCM_JLCPCB:R_0402, F.Cu at (167.5, 97.4)
- added FB6: ~, PCM_JLCPCB:R_0402, F.Cu at (33.8, 91.9)
- added FB7: ~, PCM_JLCPCB:R_0402, F.Cu at (33.8, 94.5)
- added FB8: ~, PCM_JLCPCB:R_0402, F.Cu at (169.7, 62.6)
- added H4: MountingHole, MountingHole:MountingHole_3.2mm_M3, F.Cu at (124.6, 126.3)
- added J3: Conn_ARM_SWD_TagConnect_TC2030-NL, Connector:Tag-Connect_TC2030-IDC-NL_2x03_P1.27mm_Vertical, F.Cu at (62.7, 108.0)
- added J4: Conn_01x02_Pin, Connector_PinHeader_2.54mm:PinHeader_1x02_P2.54mm_Vertical, F.Cu at (95.2, 22.8)
- added L1: MWSA1004S-220MT, easyeda2kicad:IND-SMD_L11.5-W10.0_FXL1040, F.Cu at (148.5, 123.2)
- added NT3: NetTie_2, NetTie:NetTie-2_SMD_Pad0.5mm, F.Cu at (155.0, 86.0)
- added R14: 20Ω, PCM_JLCPCB:C_0402, F.Cu at (64.8, 96.8)
- added R18: 1kΩ, PCM_JLCPCB:R_0402, F.Cu at (162.3, 98.0)
- added R2: 1kΩ, PCM_JLCPCB:R_0402, F.Cu at (163.1, 62.3)
- added R20: 0Ω, PCM_JLCPCB:R_0603, F.Cu at (48.2, 78.6)
- added R26: 100kΩ, PCM_JLCPCB:R_0603, F.Cu at (174.2, 57.0)
- added R27: 4.22kΩ, PCM_JLCPCB:R_0603, F.Cu at (172.6, 55.7)
- added R28: 100kΩ, PCM_JLCPCB:R_0603, F.Cu at (51.8, 71.8)
- added R29: 4.22kΩ, PCM_JLCPCB:R_0603, F.Cu at (51.8, 74.1)
- added R30: 1mΩ 3W, easyeda2kicad:R2512, B.Cu at (179.6, 80.7)
- added R31: 100kΩ, PCM_JLCPCB:R_0603, F.Cu at (172.8, 75.7)
- added R32: 4.22kΩ, PCM_JLCPCB:R_0603, F.Cu at (171.1, 74.4)
- added R35: 4.7kΩ, PCM_JLCPCB:R_0402, F.Cu at (53.0, 37.0)
- added R36: 4.7kΩ, PCM_JLCPCB:R_0402, F.Cu at (53.0, 38.9)
- added R37: 100kΩ, PCM_JLCPCB:R_0603, F.Cu at (172.0, 91.8)
- added R38: 4.22kΩ, PCM_JLCPCB:R_0603, F.Cu at (170.2, 90.5)
- added R39: 1mΩ 3W, easyeda2kicad:R2512, F.Cu at (169.8, 113.5)
- added R42: 3Ω, PCM_JLCPCB:R_0402, B.Cu at (173.7, 89.9)
- added R43: 10kΩ, PCM_JLCPCB:R_0402, F.Cu at (53.0, 44.4)
- added R44: 10kΩ, PCM_JLCPCB:R_0402, F.Cu at (53.0, 46.2)
- added R45: 10kΩ, PCM_JLCPCB:R_0402, F.Cu at (53.0, 48.1)
- added R46: 10kΩ, PCM_JLCPCB:R_0402, F.Cu at (53.0, 50.0)
- added R47: 120Ω, PCM_JLCPCB:R_0402, F.Cu at (89.8, 22.8)
- added R48: 10kΩ, PCM_JLCPCB:R_0603, F.Cu at (150.8, 114.8)
- added R49: 42.2kΩ, PCM_JLCPCB:R_0603, F.Cu at (161.4, 114.9)
- added R50: 10kΩ, PCM_JLCPCB:R_0402, F.Cu at (55.9, 29.6)
- added R51: 100kΩ, PCM_JLCPCB:R_0402, F.Cu at (55.9, 31.4)
- added R52: 10kΩ, PCM_JLCPCB:R_0402, F.Cu at (55.9, 33.3)
- added R53: 10Ω, PCM_JLCPCB:R_0402, F.Cu at (173.2, 77.3)
- added R54: 10Ω, PCM_JLCPCB:R_0402, F.Cu at (173.2, 78.2)
- added R55: 10Ω, PCM_JLCPCB:R_0402, F.Cu at (174.6, 58.7)
- added R56: 10Ω, PCM_JLCPCB:R_0402, F.Cu at (174.6, 59.6)
- added R57: 10Ω, PCM_JLCPCB:R_0402, F.Cu at (172.4, 93.5)
- added R58: 10Ω, PCM_JLCPCB:R_0402, F.Cu at (172.4, 94.4)
- added R59: 20Ω, PCM_JLCPCB:C_0402, B.Cu at (170.5, 69.2)
- added R60: 20Ω, PCM_JLCPCB:C_0402, F.Cu at (64.9, 94.8)
- added R61: 20Ω, PCM_JLCPCB:C_0402, F.Cu at (55.9, 50.0)
- added R62: 20Ω, PCM_JLCPCB:C_0402, F.Cu at (55.9, 51.8)
- added R63: 20Ω, PCM_JLCPCB:C_0402, F.Cu at (58.7, 29.6)
- added R64: 20Ω, PCM_JLCPCB:C_0402, F.Cu at (58.7, 31.4)
- added R65: 20Ω, PCM_JLCPCB:C_0402, F.Cu at (158.5, 95.1)
- added R66: 20Ω, PCM_JLCPCB:C_0402, F.Cu at (157.2, 79.4)
- added R67: 20Ω, PCM_JLCPCB:C_0402, F.Cu at (157.3, 60.2)
- added R68: 20Ω, PCM_JLCPCB:C_0402, F.Cu at (158.5, 91.4)
- added R69: 20Ω, PCM_JLCPCB:C_0402, F.Cu at (157.1, 75.4)
- added R7: 1kΩ, PCM_JLCPCB:R_0402, F.Cu at (162.2, 81.8)
- added R70: 20Ω, PCM_JLCPCB:C_0402, F.Cu at (157.3, 57.0)
- added R71: 3Ω, PCM_JLCPCB:R_0402, B.Cu at (173.2, 106.3)
- added R72: 20Ω, PCM_JLCPCB:C_0402, F.Cu at (165.3, 66.0)
- added R73: 10Ω, PCM_JLCPCB:R_0402, F.Cu at (81.3, 59.4)
- added R74: 10Ω, PCM_JLCPCB:R_0402, F.Cu at (84.1, 48.3)
- added R75: 20Ω, PCM_JLCPCB:C_0402, F.Cu at (163.6, 85.1)
- added R76: 20Ω, PCM_JLCPCB:C_0402, F.Cu at (163.7, 101.6)
- added R77: 20Ω, PCM_JLCPCB:C_0402, F.Cu at (65.5, 99.0)
- added R9: 20Ω, PCM_JLCPCB:C_0402, B.Cu at (169.2, 104.1)
- added S1: Tactile Button, 160gf, PCM_JLCPCB:SW_TS-1088-AR02016, F.Cu at (66.6, 73.3)
- added S2: Tactile Button, 160gf, PCM_JLCPCB:SW_TS-1088-AR02016, F.Cu at (66.6, 77.8)
- added U13: LMG2100R044RARR, easyeda2kicad:QFN-17_L5.5-W4.5-P0.50-TL_LMG2100R044, B.Cu at (173.9, 101.8)
- added U14: INA241A3xDDF, Package_TO_SOT_SMD:SOT-23-8, F.Cu at (170.6, 59.1)
- added U15: INA241A3xDDF, Package_TO_SOT_SMD:SOT-23-8, F.Cu at (169.2, 77.8)
- added U16: INA241A3xDDF, Package_TO_SOT_SMD:SOT-23-8, F.Cu at (168.4, 94.0)
- added U17: INA241A3xDDF, Package_TO_SOT_SMD:SOT-23-8, F.Cu at (161.5, 109.7)
- added U18: REF3333AIDBZR, easyeda2kicad:SOT-23-3_L2.9-W1.6-P1.90-LS2.8-BR, F.Cu at (149.8, 81.5)
- added U19: XY130-9.5-3P, easyeda2kicad:CONN-TH_XY130-9.5-3P, F.Cu at (189.3, 80.6)
- added U2: LM66200DRLR, easyeda2kicad:SOT-583-8_L2.1-W1.2-P0.50-LS1.6-BL, F.Cu at (35.3, 73.4)
- added U20: USBLC6-2P6, Package_TO_SOT_SMD:SOT-666, F.Cu at (141.0, 62.2)
- added U21: TLV7041DBV, Package_TO_SOT_SMD:SOT-23-5, F.Cu at (161.3, 84.8)
- added U22: TLV7041DBV, Package_TO_SOT_SMD:SOT-23-5, F.Cu at (161.4, 101.0)
- added U3: TCAN1044VDRBRQ1, easyeda2kicad:VSON-8_L3.0-W3.0-P0.65-BR-EP, F.Cu at (91.5, 28.0)
- added U7: S3B-PH-K-S-, easyeda2kicad:CONN-TH_3P-P2.00_S3B-PH-K-S-LF-SN, F.Cu at (91.6, 18.8)
- C1, C4: value 10pF -> 47pF; footprint PCM_JLCPCB:C_0603 -> PCM_JLCPCB:C_0402; moved to B.Cu
- C10: value 1uF -> 220nF; moved to B.Cu
- C11, C8: value 2.2nF -> 220nF; footprint PCM_JLCPCB:C_0603 -> PCM_JLCPCB:C_0805; moved to B.Cu
- C12: value 2.2nF -> 1uF; footprint PCM_JLCPCB:C_0603 -> PCM_JLCPCB:C_0805
- C13, C20, C23: value 100nF -> 1uF; footprint PCM_JLCPCB:C_0603 -> PCM_JLCPCB:C_0402
- C14: value 10uF -> 4.7uF; footprint PCM_JLCPCB:C_0603 -> PCM_JLCPCB:C_0402
- C15, C16, C17, C18, C21, C28, C3, C45, C46, C6: footprint PCM_JLCPCB:C_0603 -> PCM_JLCPCB:C_0402
- C19: value 100nF -> 1uF; footprint PCM_JLCPCB:C_0603 -> PCM_JLCPCB:C_0805
- C2: value 2.2uF -> 100nF; footprint PCM_JLCPCB:C_0603 -> PCM_JLCPCB:C_0402
- C22, C26, C9: value 1uF -> 100nF; footprint PCM_JLCPCB:C_0603 -> PCM_JLCPCB:C_0402
- C25: value 2.2uF -> 47pF; footprint PCM_JLCPCB:C_0603 -> PCM_JLCPCB:C_0402; moved to B.Cu
- C27: value 47nF -> 100nF; footprint PCM_JLCPCB:C_0603 -> PCM_JLCPCB:C_0402
- C29: value VEJ331M2ATR-1816 -> 1uF; footprint footprints:VEJ331M2ATR-1816 -> PCM_JLCPCB:C_0402
- C31: value 2.2nF -> 47pF; footprint PCM_JLCPCB:C_0603 -> PCM_JLCPCB:C_0402; moved to B.Cu
- C32: value VEJ331M2ATR-1816 -> 100nF; footprint footprints:VEJ331M2ATR-1816 -> PCM_JLCPCB:C_0402
- C34: value 58pF -> 100nF; footprint PCM_JLCPCB:C_0603 -> PCM_JLCPCB:C_0402
- C36: value 2.2nF -> 1uF; footprint PCM_JLCPCB:C_0603 -> PCM_JLCPCB:C_0402
- C39: value 22uF -> 1uF; footprint PCM_JLCPCB:C_0603 -> PCM_JLCPCB:C_0402
- C41, C44: value 22uF -> 220nF; footprint PCM_JLCPCB:C_0603 -> PCM_JLCPCB:C_0805; moved to B.Cu
- C5: footprint PCM_JLCPCB:C_0603 -> PCM_JLCPCB:C_0402; moved to B.Cu
- C7: value 2.2nF -> 100nF; footprint PCM_JLCPCB:C_0603 -> PCM_JLCPCB:C_0402
- J2: footprint footprints:AMASS_XT60PW-M -> easyeda2kicad:AMASS_XT60PW-M
- R1: value 3.3Ω -> 10kΩ; footprint PCM_JLCPCB:R_0603 -> PCM_JLCPCB:R_0402
- R10: value 100kΩ -> 220Ω; footprint PCM_JLCPCB:R_0603 -> PCM_JLCPCB:R_0402
- R11: value 383kΩ -> 40.2kΩ; footprint PCM_JLCPCB:R_0805 -> PCM_JLCPCB:R_0603
- R12: value 9.76kΩ -> 20kΩ; footprint PCM_JLCPCB:R_0805 -> PCM_JLCPCB:R_0402
- R13: value 10kΩ -> 220Ω; footprint PCM_JLCPCB:R_0603 -> PCM_JLCPCB:R_0402
- R15: value 150kΩ -> 5.1kΩ; footprint PCM_JLCPCB:R_0603 -> PCM_JLCPCB:R_0402
- R16, R6: footprint PCM_JLCPCB:R_0603 -> PCM_JLCPCB:R_0402
- R17: value 5.1kΩ -> 100kΩ; footprint PCM_JLCPCB:R_0603 -> PCM_JLCPCB:R_0402
- R19: value 360kΩ -> 0Ω
- R21: value 470kΩ -> 1mΩ 3W; footprint PCM_JLCPCB:R_0603 -> easyeda2kicad:R2512; moved to B.Cu
- R22: value 330Ω -> 220Ω; footprint PCM_JLCPCB:R_0603 -> PCM_JLCPCB:R_0402
- R23: value 330Ω -> 120Ω; footprint PCM_JLCPCB:R_0603 -> PCM_JLCPCB:R_0402
- R24: value 4.7kΩ -> 3Ω; footprint PCM_JLCPCB:R_0603 -> PCM_JLCPCB:R_0402; moved to B.Cu
- R25: value 4.7kΩ -> 20kΩ; footprint PCM_JLCPCB:R_0603 -> PCM_JLCPCB:R_0402
- R3: value 3.3Ω -> 20kΩ; footprint PCM_JLCPCB:R_0603 -> PCM_JLCPCB:R_0402
- R34: value 2.7Ω -> 1mΩ 3W; footprint PCM_JLCPCB:R_0805 -> easyeda2kicad:R2512; moved to B.Cu
- R4: value 2.7Ω -> 20Ω; footprint PCM_JLCPCB:R_0805 -> PCM_JLCPCB:C_0402; moved to B.Cu
- R5: value 2.7Ω -> 20Ω; footprint PCM_JLCPCB:R_0805 -> PCM_JLCPCB:C_0402
- R8: value 330kΩ -> 10kΩ; footprint PCM_JLCPCB:R_0603 -> PCM_JLCPCB:R_0402
- U1: value UCC27211ADRMR -> LMG2100R044RARR; footprint easyeda2kicad:VSON-8_L4.0-W4.0-P0.80-TL-EP -> easyeda2kicad:QFN-17_L5.5-W4.5-P0.50-TL_LMG2100R044; moved to B.Cu
- U10: moved to B.Cu
- U11: value USBLC6-2P6 -> TLV7041DBV; footprint Package_TO_SOT_SMD:SOT-666 -> Package_TO_SOT_SMD:SOT-23-5
- U12: value MR60PW-M.G.B -> LMR38010FDDAR; footprint footprints:CONN-TH_MR60PW -> easyeda2kicad:ESOP-8_L4.9-W3.9-P1.27-LS6.0-BL-EP3.1
- U5: value INA240A2D -> TPD2E2U06DCK; footprint Package_SO:SOIC-8_3.9x4.9mm_P1.27mm -> Package_TO_SOT_SMD:SOT-323_SC-70
- U8: value LM5164DDA -> LMG2100R044RARR; footprint Package_SO:HSOP-8-1EP_3.9x4.9mm_P1.27mm_EP2.41x3.1mm_ThermalVias -> easyeda2kicad:QFN-17_L5.5-W4.5-P0.50-TL_LMG2100R044; moved to B.Cu
- X1: value X322516MLB4SI -> X322524MOB4SI; footprint PCM_JLCPCB:OSC-SMD_4P-L3.2-W2.5-BL -> easyeda2kicad:CRYSTAL-SMD_4P-L3.2-W2.5-BL
- moved C32 160.9 mm to (41.6, 40.7)
- moved C29 141.3 mm to (41.6, 35.1)
- moved D1 131.5 mm to (26.1, 65.3)
- moved D2 131.5 mm to (26.1, 68.3)
- moved U4 126.8 mm to (30.9, 74.3)
- moved R22 119.0 mm to (53.0, 29.6)
- moved R23 114.3 mm to (53.0, 31.4)
- moved FB2 112.7 mm to (21.8, 67.5)
- moved FB1 112.7 mm to (21.8, 65.0)
- moved R5 111.1 mm to (50.2, 33.3)
- moved R6 111.0 mm to (50.2, 35.1)
- moved R8 110.2 mm to (50.2, 38.9)
- moved R13 109.6 mm to (50.2, 44.4)
- moved R10 109.4 mm to (50.2, 42.5)
- moved C45 106.4 mm to (44.5, 31.4)
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Connections:
- C1 pad 1: /HSE_IN -> /HIB
- C10 pad 2: GND -> PGND
- C11 pad 1: Net-(C11-Pad1) -> VM
- C11 pad 2: Net-(C11-Pad2) -> PGND
- C12 pad 1: Net-(C11-Pad2) -> VM
- C12 pad 2: Net-(C12-Pad2) -> PGND
- C13 pad 1: /NRST -> 5V_OR
- C14 pad 1: GND -> +3V3
- C14 pad 2: +3V3 -> GND
- C19 pad 1: +3V3 -> VM
- C19 pad 2: GND -> PGND
- C2 pad 1: +12V_VM -> GND
- C2 pad 2: GND -> Net-(U16-V+)
- C21 pad 1: +3V3A -> +3V3
- C23 pad 1: +3V3 -> +3V3A
- C25 pad 1: VM -> /HIA
- C26 pad 1: +3V3 -> /AMB_TMP
- C27 pad 1: /VSENVM -> VREF
- C28 pad 1: +3V3 -> /PHASE_TMP
- C29 pad 1: VM -> /REFIN
- C3 pad 1: +12V_VM -> VREF
- C31 pad 1: /SW_12V -> /HIC
- C31 pad 2: Net-(U8-BST) -> GND
- C32 pad 1: VM -> VREF
- C34 pad 1: Net-(C34-Pad1) -> Net-(U15-V+)
- C34 pad 2: /FB_12V -> GND
- C36 pad 1: Net-(C34-Pad1) -> VBUCK
- C36 pad 2: +12V_VM -> GND
- C39 pad 1: +12V_VM -> +5V_USB
- C4 pad 1: /HSE_IN -> /LIB
- C41 pad 1: +12V_VM -> VM
- C41 pad 2: GND -> PGND
- C44 pad 1: +12V_VM -> VM
- C44 pad 2: GND -> PGND
- C45 pad 1: /PHASE_TMP -> +3V3
- C46 pad 1: /AMB_TMP -> GND
- C46 pad 2: GND -> Net-(U17-V+)
- C5 pad 1: Net-(U1-HS) -> VBUCK
- C5 pad 2: Net-(U1-HB) -> GND
- C6 pad 1: +5V_USB -> +3V3
- C7 pad 1: /GHA -> VREF
- C7 pad 2: /MP_A -> GND
- C8 pad 1: /GLA -> VM
- C8 pad 2: GND -> PGND
- J1 pad A5: Net-(J1-CC1) -> /CC1
- J1 pad A6: Net-(J1-D+-PadA6) -> /D+
- J1 pad A7: Net-(J1-D--PadA7) -> /D-
- J1 pad B5: Net-(J1-CC2) -> /CC2
- J1 pad B6: Net-(J1-D+-PadA6) -> /D+
- J1 pad B7: Net-(J1-D--PadA7) -> /D-
- J2 pad 1: VM -> VDC
- J2 pad 2: GND -> PGND
- J2 pad SH1: GND -> PGND
- J2 pad SH2: GND -> PGND
- R1 pad 1: /GLA -> +3V3
- R1 pad 2: Net-(U1-LO) -> /OCP
- R10 pad 1: /RON_12V -> Net-(D4-Pad1)
- R11 pad 1: VM -> /FB
- R11 pad 2: /VSENVM -> VBUCK
- R12 pad 1: /VSENVM -> Net-(U21--)
- R13 pad 1: +3V3 -> Net-(D1-Pad1)
- R13 pad 2: Net-(U10-~{CS}) -> GND
- R15 pad 1: /FB_12V -> /CC1
- R16 pad 1: GND -> /CC2
- R16 pad 2: Net-(J1-CC2) -> GND
- R17 pad 1: GND -> +3V3
- R17 pad 2: Net-(J1-CC1) -> /ST
- R19 pad 1: /SW_12V -> PGND
- R19 pad 2: Net-(C34-Pad1) -> GND
- R21 pad 1: /FB_12V -> CSA+
- R21 pad 2: +12V_VM -> CSA-
- R22 pad 1: Net-(D1-Pad1) -> Net-(D2-Pad1)
- R23 pad 1: Net-(D2-Pad1) -> Net-(D5-Pad1)
- R24 pad 1: +3V3 -> Net-(C99-Pad1)
- R24 pad 2: /PHASE_TMP -> /HBA
- R25 pad 1: +3V3 -> Net-(U22--)
- R25 pad 2: /AMB_TMP -> GND
- R3 pad 1: Net-(U1-HO) -> Net-(U11--)
- R3 pad 2: /GHA -> GND
- R34 pad 1: /MP_A -> CSC+
- R34 pad 2: /MOTA -> CSC-
- R4 pad 1: VM -> /HIB
- R4 pad 2: Net-(C11-Pad1) -> /INHB
- R5 pad 1: Net-(C12-Pad2) -> /LIB
- R5 pad 2: GND -> /INLB
- R6 pad 2: /SW_BOOT0 -> GND
- R8 pad 1: /EN_12V -> +3V3
- R8 pad 2: GND -> /ENC_CS
- U1 pad 1: +12V_VM -> unconnected-(U1-NC-Pad1)
- U1 pad 2: Net-(U1-HB) -> unconnected-(U1-NC-Pad2)
- U1 pad 3: Net-(U1-HO) -> unconnected-(U1-NC-Pad3)
- U1 pad 4: Net-(U1-HS) -> unconnected-(U1-NC-Pad4)
- U1 pad 5: /PWM_HA -> CSA+
- U1 pad 6: /PWM_LA -> PGND
- U1 pad 7: GND -> VM
- U1 pad 8: Net-(U1-LO) -> unconnected-(U1-NC-Pad8)
- U1 pad 9: GND -> unconnected-(U1-NC-Pad9)
- U10 pad 1: Net-(U10-~{CS}) -> /ENC_CS
- U10 pad 12: unconnected-(U10-VDD3V3-Pad12) -> Net-(U10-VDD3V3)
- U10 pad 2: unconnected-(U10-CLK-Pad2) -> /SPI_SCK
- U10 pad 3: unconnected-(U10-MISO-Pad3) -> /SPI_MISO
- U10 pad 4: unconnected-(U10-MOSI-Pad4) -> /SPI_MOSI
- U11 pad 1: Net-(J1-D--PadA7) -> /OCP
- U11 pad 3: Net-(J1-D+-PadA6) -> Net-(U11-+)
- U11 pad 4: /USB_D+ -> Net-(U11--)
- U11 pad 5: /USB_VBUS -> +3V3
- U12 pad 1: /MOTA -> GND
- U12 pad 2: /MOTB -> VDC
- U12 pad 3: /MOTC -> VDC
- U12 pad 4: GND -> /RT
- U12 pad 5: GND -> /FB
- U4 pad 1: +5V_USB -> 5V_OR
- U4 pad 3: +5V_USB -> 5V_OR
- U5 pad 1: /MP_A -> /CANH
- U5 pad 2: GND -> /CANL
- U5 pad 3: +3V3 -> GND
- U6 pad 10: unconnected-(U6-PC2-Pad10) -> /AMB_TMP_ADC
- U6 pad 11: unconnected-(U6-PC3-Pad11) -> /PHASE_TMP_ADC
- U6 pad 12: /VSENVM -> unconnected-(U6-PA0-Pad12)
- U6 pad 13: /PHASE_TMP -> /ENC_CS
- U6 pad 14: /AMB_TMP -> unconnected-(U6-PA2-Pad14)
- U6 pad 17: /CSA -> unconnected-(U6-PA3-Pad17)
- U6 pad 19: unconnected-(U6-PA5-Pad19) -> /SPI_SCK
- U6 pad 20: unconnected-(U6-PA6-Pad20) -> /SPI_MISO
- U6 pad 21: /CSB -> /SPI_MOSI
- U6 pad 24: /CSC -> /IC_ADC
- U6 pad 25: unconnected-(U6-PB1-Pad25) -> /IB_ADC
- U6 pad 26: unconnected-(U6-PB2-Pad26) -> /IA_ADC
- U6 pad 28: unconnected-(U6-VREF+-Pad28) -> +3V3A
- U6 pad 33: unconnected-(U6-PB11-Pad33) -> Net-(U6-PB11)
- U6 pad 35: /PWM_LA -> /VC_ADC
- U6 pad 36: /PWM_LB -> /VB_ADC
- U6 pad 37: /PWM_LC -> /VA_ADC
- U6 pad 38: unconnected-(U6-PC6-Pad38) -> /INLC
- U6 pad 39: unconnected-(U6-PC7-Pad39) -> /INHC
- U6 pad 40: unconnected-(U6-PC8-Pad40) -> /INLB
- U6 pad 41: unconnected-(U6-PC9-Pad41) -> /INHB
- U6 pad 42: /PWM_HA -> /INLA
- U6 pad 43: /PWM_HB -> /INHA
- U6 pad 44: /PWM_HC -> unconnected-(U6-PA10-Pad44)
- U6 pad 49: /SWCLK -> /SWDIO
- U6 pad 50: /CAN_TX -> /SWCLK
- U6 pad 52: /SPI_MOSI -> unconnected-(U6-PC10-Pad52)
- U6 pad 53: /SPI_MISO -> /HEARBEAT
- U6 pad 54: /SPI_SCK -> /FAULT
- U6 pad 56: /CAN_RX -> /SWO
- U6 pad 57: /CAN_TX -> unconnected-(U6-PB4-Pad57)
- U6 pad 58: unconnected-(U6-PB5-Pad58) -> /CAN_RX
- U6 pad 59: unconnected-(U6-PB6-Pad59) -> /CAN_TX
- U6 pad 8: unconnected-(U6-PC0-Pad8) -> /IDC_ADC
- U6 pad 9: unconnected-(U6-PC1-Pad9) -> /VDC_ADC
- U8 pad 1: GND -> unconnected-(U8-NC-Pad1)
- U8 pad 2: VM -> unconnected-(U8-NC-Pad2)
- U8 pad 3: /EN_12V -> unconnected-(U8-NC-Pad3)
- U8 pad 4: /RON_12V -> unconnected-(U8-NC-Pad4)
- U8 pad 5: /FB_12V -> CSB+
- U8 pad 6: unconnected-(U8-PGOOD-Pad6) -> PGND
- U8 pad 7: Net-(U8-BST) -> VM
- U8 pad 8: /SW_12V -> unconnected-(U8-NC-Pad8)
- U8 pad 9: GND -> unconnected-(U8-NC-Pad9)
- X1 pad 1: /HSE_IN -> /HSE_OUT
Routing:
- net GND: track 0.00 -> 33.6 mm, vias 0 -> 3
- net /USB_D+: track 0.00 -> 30.6 mm
- net /USB_D-: track 0.00 -> 30.5 mm
- net CSC-: track 0.00 -> 24.7 mm, vias 0 -> 2
- net CSB-: track 0.00 -> 24.2 mm, vias 0 -> 2
- net CSA-: track 0.00 -> 22.2 mm, vias 0 -> 2
- net /VSENA: track 0.00 -> 18.8 mm
- net /VSENB: track 0.00 -> 18.1 mm
- net /IA: track 0.00 -> 18.1 mm
- net /IB: track 0.00 -> 17.0 mm
- net /IC: track 0.00 -> 15.5 mm
- net /VSENC: track 0.00 -> 15.4 mm
- net CSB+: track 0.00 -> 11.7 mm, vias 0 -> 1
- net CSC+: track 0.00 -> 11.0 mm, vias 0 -> 1
- net +3V3: track 0.00 -> 10.7 mm
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- added copper zone on B.Cu, net CSA+
- added copper zone on B.Cu, net CSB+
- added copper zone on B.Cu, net CSB-
- added copper zone on B.Cu, net CSC+
- added copper zone on B.Cu, net VM
- added copper zone on F.Cu, net VM
Other:
- board size 80 x 80 mm -> 77 x 80 mm
