File: bench_stm32_esc/bench_stm32_esc.kicad_pcb (KiCad board)
At the start: 4 copper layers, 117 x 75 mm, 108 parts, among them CN1 S6B-PH-K-S-, CN10 Conn_02x19_Odd_Even, CN7 Conn_02x19_Odd_Even, J1 XT60PW-M, J2 Conn_ST_STDC14, Q1 CSD19532Q5B, Q2 CSD19532Q5B, Q3 CSD19532Q5B, Q4 CSD19532Q5B, Q5 CSD19532Q5B, Q6 CSD19532Q5B, U1 DRV8353RSRGZT, U2 AMS1117, U3 TPD1E05U06DYA, U4 MR60PW-M.G.B, U7 TB60

Commit message: Revision 1.1
Parts:
- removed C16: VT10UF100V167RV0127, footprints:VT10UF100V167RV0127
- removed C34, C35: 2.2nF, PCM_JLCPCB:C_0603
- removed CN10, CN7: Conn_02x19_Odd_Even, Connector_PinSocket_2.54mm:PinSocket_2x19_P2.54mm_Vertical
- removed TP2, TP3, TP4, TP5: TestPoint, TestPoint:TestPoint_Pad_1.5x1.5mm
- added C41: 100nF, PCM_JLCPCB:C_0402, B.Cu at (151.8, 49.1)
- added C42: 1uF, PCM_JLCPCB:C_0402, F.Cu at (147.5, 81.4)
- added C43: 1uF, PCM_JLCPCB:C_0402, F.Cu at (150.0, 77.0)
- added C44: 4.7uF, PCM_JLCPCB:C_0402, F.Cu at (160.0, 48.8)
- added C45: 1uF, PCM_JLCPCB:C_0402, F.Cu at (156.9, 59.8)
- added C46: 100nF, PCM_JLCPCB:C_0402, F.Cu at (144.7, 56.0)
- added C47: 100nF, PCM_JLCPCB:C_0402, F.Cu at (156.3, 59.2)
- added C48: 100nF, PCM_JLCPCB:C_0402, F.Cu at (159.1, 48.8)
- added C49: 100nF, PCM_JLCPCB:C_0402, F.Cu at (147.3, 46.0)
- added C50: 100nF, PCM_JLCPCB:C_0402, F.Cu at (144.3, 54.6)
- added C51: 1nF, PCM_JLCPCB:C_0402, B.Cu at (146.3, 50.9)
- added C52: 1uF, PCM_JLCPCB:C_0402, F.Cu at (143.9, 53.3)
- added C53: 100nF, PCM_JLCPCB:C_0402, F.Cu at (143.8, 56.0)
- added C54: 2.2uF, PCM_JLCPCB:C_0402, F.Cu at (140.0, 81.0)
- added C55: 2.2uF, PCM_JLCPCB:C_0402, F.Cu at (144.2, 81.0)
- added C56: 10nF, PCM_JLCPCB:C_0402, B.Cu at (151.2, 56.0)
- added C57: 10nF, PCM_JLCPCB:C_0402, B.Cu at (148.8, 55.2)
- added C58: 10nF, PCM_JLCPCB:C_0402, B.Cu at (147.0, 55.3)
- added C61: 47nF, PCM_JLCPCB:C_0402, B.Cu at (182.9, 42.2)
- added C62: 47nF, PCM_JLCPCB:C_0402, B.Cu at (178.6, 43.0)
- added C63: 47nF, PCM_JLCPCB:C_0402, B.Cu at (173.4, 44.0)
- added C64: 100nF, PCM_JLCPCB:C_0402, F.Cu at (149.4, 43.4)
- added C65: 100nF, PCM_JLCPCB:C_0402, B.Cu at (150.2, 49.1)
- added C66: 1nF, PCM_JLCPCB:C_0402, B.Cu at (148.1, 50.9)
- added C67: 1nF, PCM_JLCPCB:C_0402, B.Cu at (150.0, 50.9)
- added C68: 4.7uF, PCM_JLCPCB:C_1206, B.Cu at (182.2, 51.8)
- added C69: 4.7uF, PCM_JLCPCB:C_1206, B.Cu at (182.3, 63.8)
- added C70: 4.7uF, PCM_JLCPCB:C_1206, B.Cu at (182.1, 75.9)
- added C71: 4.7uF, PCM_JLCPCB:C_1206, B.Cu at (182.1, 73.6)
- added C72: 4.7uF, PCM_JLCPCB:C_1206, B.Cu at (182.3, 61.5)
- added C73: 4.7uF, PCM_JLCPCB:C_1206, B.Cu at (182.2, 49.4)
- added C76: 100nF, PCM_JLCPCB:C_0402, F.Cu at (163.9, 44.1)
- added C83: 100nF, PCM_JLCPCB:C_0402, F.Cu at (144.8, 53.3)
- added C85: 18pF, PCM_JLCPCB:C_0402, F.Cu at (151.1, 43.4)
- added C87: 18pF, PCM_JLCPCB:C_0402, F.Cu at (155.9, 43.3)
- added C93: 1uF, PCM_JLCPCB:C_0402, F.Cu at (154.6, 74.5)
- added CN2: 1053141104, easyeda2kicad:CONN-TH_4P-P2.50_MOLEX_1053141104, F.Cu at (139.3, 74.1)
- added CN3: 1053141104, easyeda2kicad:CONN-TH_4P-P2.50_MOLEX_1053141104, F.Cu at (139.3, 61.3)
- added D3: PESD2CAN,215, easyeda2kicad:SOT-23-3_L2.9-W1.3-P1.90-LS2.4-BR, B.Cu at (143.2, 71.0)
- added FB1: ~, PCM_JLCPCB:FB_0603, F.Cu at (142.6, 54.6)
- added FB2: ~, PCM_JLCPCB:FB_0603, F.Cu at (142.0, 80.5)
- added J3: Conn_ARM_SWD_TagConnect_TC2030-NL, Connector:Tag-Connect_TC2030-IDC-NL_2x03_P1.27mm_Vertical, F.Cu at (164.1, 55.8)
- added J4: Screw_Terminal_01x05, footprints:CUI_TB005_-762-05BE, F.Cu at (197.7, 84.0)
- added R20: 56Ω, PCM_JLCPCB:R_0402, B.Cu at (152.1, 56.0)
- added R23: 100kΩ, PCM_JLCPCB:R_0402, F.Cu at (149.8, 79.8)
- added R29: 5.1kΩ, PCM_JLCPCB:R_0402, F.Cu at (136.4, 84.7)
- added R30: 5.1kΩ, PCM_JLCPCB:R_0402, F.Cu at (136.4, 81.5)
- added R31: 10Ω, PCM_JLCPCB:R_0402, B.Cu at (187.7, 67.1)
- added R32: 10Ω, PCM_JLCPCB:R_0402, B.Cu at (187.1, 79.0)
- added R33: 383kΩ, PCM_JLCPCB:R_0402, B.Cu at (187.4, 42.6)
- added R34: 1kΩ, PCM_JLCPCB:R_0402, B.Cu at (149.1, 50.9)
- added R35: 383kΩ, PCM_JLCPCB:R_0402, B.Cu at (187.4, 43.5)
- added R36: 1kΩ, PCM_JLCPCB:R_0402, B.Cu at (147.2, 50.9)
- added R37: 383kΩ, PCM_JLCPCB:R_0402, B.Cu at (187.4, 44.4)
- added R38: 9.76kΩ, PCM_JLCPCB:R_0402, B.Cu at (174.3, 44.0)
- added R39: 9.76kΩ, PCM_JLCPCB:R_0402, B.Cu at (179.4, 43.0)
- added R40: 9.76kΩ, PCM_JLCPCB:R_0402, B.Cu at (182.1, 42.2)
- added R41: 1kΩ, PCM_JLCPCB:R_0402, B.Cu at (145.4, 50.9)
- added R42: 100Ω, PCM_JLCPCB:R_0402, F.Cu at (175.0, 67.1)
- added R43: 10kΩ, PCM_JLCPCB:R_0402, F.Cu at (167.0, 57.5)
- added R44: 100Ω, PCM_JLCPCB:R_0402, F.Cu at (175.0, 68.0)
- added R45: 100Ω, PCM_JLCPCB:R_0402, F.Cu at (174.8, 61.7)
- added R46: 100Ω, PCM_JLCPCB:R_0402, F.Cu at (174.2, 61.0)
- added R47: 100Ω, PCM_JLCPCB:R_0402, B.Cu at (152.7, 49.1)
- added R48: 100Ω, PCM_JLCPCB:R_0402, F.Cu at (150.2, 43.4)
- added R49: 100Ω, PCM_JLCPCB:R_0402, B.Cu at (151.0, 49.1)
- added R50: 10kΩ, PCM_JLCPCB:R_0402, B.Cu at (141.8, 45.3)
- added R51: 100kΩ, PCM_JLCPCB:R_0402, F.Cu at (149.2, 83.4)
- added R52: 20kΩ, PCM_JLCPCB:R_0402, B.Cu at (141.8, 43.5)
- added R53: 10kΩ, PCM_JLCPCB:R_0402, B.Cu at (143.5, 46.2)
- added R54: 20kΩ, PCM_JLCPCB:R_0402, B.Cu at (143.5, 44.4)
- added R55: 1kΩ, PCM_JLCPCB:R_0402, B.Cu at (162.1, 58.8)
- added R56: 100Ω, PCM_JLCPCB:R_0402, F.Cu at (143.2, 50.4)
- added S1: Tactile Button, 160gf, PCM_JLCPCB:SW_TS-1088-AR02016, F.Cu at (163.9, 46.2)
- added S2: Tactile Button, 160gf, PCM_JLCPCB:SW_TS-1088-AR02016, F.Cu at (163.9, 49.7)
- added TP10: TestPoint, TestPoint:TestPoint_Pad_1.5x1.5mm, B.Cu at (178.6, 62.6)
- added TP11: TestPoint, TestPoint:TestPoint_Pad_1.5x1.5mm, B.Cu at (178.4, 74.8)
- added TP12: TestPoint, TestPoint:TestPoint_Pad_1.5x1.5mm, F.Cu at (154.0, 80.2)
- added TP13: TestPoint, TestPoint:TestPoint_Pad_1.5x1.5mm, F.Cu at (158.2, 75.0)
- added TP9: TestPoint, TestPoint:TestPoint_Pad_1.5x1.5mm, B.Cu at (178.4, 50.6)
- added U20: USBLC6-2P6, Package_TO_SOT_SMD:SOT-666, F.Cu at (138.5, 82.8)
- added U5: LM66200DRLR, easyeda2kicad:SOT-583-8_L2.1-W1.2-P0.50-LS1.6-BL, F.Cu at (149.2, 81.8)
- added U6: AP2112K-3.3, Package_TO_SOT_SMD:SOT-23-5, F.Cu at (153.1, 77.0)
- added U8: TCAN1462VDRBRQ1, easyeda2kicad:DFN-8_L3.0-W3.0-P0.65-TL-EP2.4, B.Cu at (134.7, 50.8)
- added X1: X322524MOB4SI, easyeda2kicad:CRYSTAL-SMD_4P-L3.2-W2.5-BL, F.Cu at (153.6, 43.4)
- C1, C2, C3, C4: value 1uF -> EEHZC1K470V; footprint PCM_JLCPCB:C_0603 -> easyeda2kicad:CAP-SMD_BD10.0-L10.3-W10.3-FD
- C10: value 1uF -> 47uF; footprint PCM_JLCPCB:C_0805 -> PCM_JLCPCB:C_1206
- C11: value 10nF -> 100nF; footprint PCM_JLCPCB:C_0603 -> PCM_JLCPCB:C_0402
- C12: value 3.3nF -> 100nF; footprint PCM_JLCPCB:C_0603 -> PCM_JLCPCB:C_0402
- C13: value 10uF -> 1uF; footprint PCM_JLCPCB:C_CASE-A-3216-18(mm) -> PCM_JLCPCB:C_0402
- C14: value 2.2uF -> 1uF; footprint PCM_JLCPCB:C_0603 -> PCM_JLCPCB:C_0402
- C15: value 22uF -> 1uF; footprint PCM_JLCPCB:C_CASE-A-3216-18(mm) -> PCM_JLCPCB:C_0402
- C17, C19: value 2.2nF -> 47uF; footprint PCM_JLCPCB:C_0603 -> PCM_JLCPCB:C_1206
- C18, C26, C32, C5: footprint PCM_JLCPCB:C_0603 -> PCM_JLCPCB:C_0402; moved to B.Cu
- C20, C22: value 2.2nF -> 100nF; footprint PCM_JLCPCB:C_0603 -> PCM_JLCPCB:C_0402
- C21, C24, C8: footprint PCM_JLCPCB:C_0603 -> PCM_JLCPCB:C_0402
- C23, C27, C28: value 2.2nF -> 1uF; footprint PCM_JLCPCB:C_0603 -> PCM_JLCPCB:C_1206
- C25: value 1uF -> 1nF; footprint PCM_JLCPCB:C_0805 -> PCM_JLCPCB:C_0402
- C29: value 2.2nF -> 1uF; footprint PCM_JLCPCB:C_0603 -> PCM_JLCPCB:C_0402; moved to B.Cu
- C30: value 1nF -> 100nF; footprint PCM_JLCPCB:C_0603 -> PCM_JLCPCB:C_0402; moved to B.Cu
- C31: value 1uF -> 100nF; footprint PCM_JLCPCB:C_0805 -> PCM_JLCPCB:C_0402; moved to B.Cu
- C33: value 2.2nF -> 100nF; footprint PCM_JLCPCB:C_0603 -> PCM_JLCPCB:C_0402; moved to B.Cu
- C36: value VEJ331M2ATR-1816 -> 1uF; footprint footprints:VEJ331M2ATR-1816 -> PCM_JLCPCB:C_0402; moved to B.Cu
- C37: value VEJ331M2ATR-1816 -> 1uF; footprint footprints:VEJ331M2ATR-1816 -> PCM_JLCPCB:C_0402
- C39, C40: value 100nF -> 2.2nF; footprint PCM_JLCPCB:C_0603 -> PCM_JLCPCB:C_0402; moved to B.Cu
- C7: value 1uF -> EEHZC1K470V; footprint PCM_JLCPCB:C_0805 -> easyeda2kicad:CAP-SMD_BD10.0-L10.3-W10.3-FD
- C9: value 100nF -> GRM32EC72A106KE05L; footprint PCM_JLCPCB:C_0603 -> easyeda2kicad:C1210
- CN1: value S6B-PH-K-S- -> 1053141104; footprint footprints:S6B-PH-K-S(LF)(SN) -> easyeda2kicad:CONN-TH_4P-P2.50_MOLEX_1053141104
- D1: value DSK120 -> White; footprint PCM_JLCPCB:D_SOD-123FL -> PCM_JLCPCB:D_0603
- J1: value XT60PW-M -> Conn_02x01; footprint footprints:AMASS_XT60PW-M -> Connector_PinHeader_2.54mm:PinHeader_2x01_P2.54mm_Vertical
- J2: value Conn_ST_STDC14 -> USB_C_Receptacle_USB2.0_16P; footprint Connector_PinHeader_1.27mm:PinHeader_2x07_P1.27mm_Vertical -> Connector_USB:USB_C_Receptacle_HRO_TYPE-C-31-M-12
- L1: value SMDRH104R-331MT -> FNR4020S8R2MT; footprint footprints:SMDRH104R-331MT -> easyeda2kicad:IND-SMD_L4.0-W4.0_FNR40XXS
- NT1, NT2, NT5, R10, R13, R7, TH1, TP1, TP6, TP7, TP8: moved to B.Cu
- Q1, Q2, Q3, Q4, Q5, Q6: value CSD19532Q5B -> IAUCN08S7N019ATMA1; moved to B.Cu
- R1: value 100kΩ -> 100Ω; footprint PCM_JLCPCB:R_0603 -> PCM_JLCPCB:R_0402
- R11: value 2.7Ω -> 19.1kΩ; footprint PCM_JLCPCB:R_0805 -> PCM_JLCPCB:R_0402
- R12, R8, R9: value 7mΩ -> 2mΩ; moved to B.Cu
- R14: value 2.7Ω -> 120Ω; footprint PCM_JLCPCB:R_0805 -> PCM_JLCPCB:R_0402; moved to B.Cu
- R15, R16: footprint PCM_JLCPCB:R_0603 -> PCM_JLCPCB:R_0402; moved to B.Cu
- R17: value 1kΩ -> 4.7kΩ; footprint PCM_JLCPCB:R_0603 -> PCM_JLCPCB:R_0402; moved to B.Cu
- R2: value 274kΩ -> 100Ω; footprint PCM_JLCPCB:R_0603 -> PCM_JLCPCB:R_0402
- R21, R24: footprint PCM_JLCPCB:R_0603 -> PCM_JLCPCB:R_0402
- R22: value 4.7kΩ -> 10kΩ; footprint PCM_JLCPCB:R_0603 -> PCM_JLCPCB:R_0402
- R25: value 10kΩ -> 10Ω; footprint PCM_JLCPCB:R_0603 -> PCM_JLCPCB:R_0402; moved to B.Cu
- R26, R27, R28: value 330Ω -> 10Ω; footprint PCM_JLCPCB:R_0603 -> PCM_JLCPCB:R_0402; moved to B.Cu
- R3, R4: value 10kΩ -> 330Ω; footprint PCM_JLCPCB:R_0603 -> PCM_JLCPCB:R_0402
- R5: value 2.2Ω -> 330Ω; footprint PCM_JLCPCB:R_0603 -> PCM_JLCPCB:R_0402
- R6: value 2.7Ω -> 100kΩ; footprint PCM_JLCPCB:R_0805 -> PCM_JLCPCB:R_0402
- U1: value DRV8353RSRGZT -> LMR51635YDDCR; footprint footprints:QFN50P700X700X100-49N -> easyeda2kicad:SOT-23-6_L2.9-W1.6-P0.95-LS2.8-BL
- U2: value AMS1117 -> MA730; footprint PCM_JLCPCB:SOT-223-3_L6.5-W3.4-P2.30-LS7.0-BR -> Package_DFN_QFN:QFN-16-1EP_3x3mm_P0.5mm_EP1.75x1.75mm; moved to B.Cu
- U4: value MR60PW-M.G.B -> DRV8353SRTAR; footprint footprints:CONN-TH_MR60PW -> easyeda2kicad:WQFN-40_L6.0-W6.0-P0.50-TL-EP4.5
- U7: value TB60 -> STM32G474RETx; footprint footprints:TB60 -> Package_QFP:LQFP-64_10x10mm_P0.5mm
- moved J2 152.4 mm to (130.2, 82.9), turned to -90 degrees
- moved H4 112.6 mm to (198.5, 93.0)
- moved C36 82.0 mm to (135.0, 47.8), turned to 90 degrees
- moved J1 78.8 mm to (134.8, 55.5), turned to 180 degrees
- moved R28 74.7 mm to (187.1, 54.6), turned to 0 degrees
- moved H3 69.8 mm to (132.0, 93.0)
- moved R16 65.7 mm to (149.7, 55.2), turned to 90 degrees
- moved R15 63.7 mm to (147.9, 55.2), turned to 90 degrees
- moved U7 61.5 mm to (151.9, 52.2), turned to -90 degrees
- moved C3 52.4 mm to (182.9, 47.2)
- moved C33 50.3 mm to (136.8, 53.0), turned to 180 degrees
- moved R22 50.1 mm to (169.3, 58.9), turned to -90 degrees
- moved R14 47.2 mm to (137.1, 55.7), turned to 180 degrees
- moved H1 45.5 mm to (132.0, 44.5)
- moved C15 44.8 mm to (165.2, 66.6), turned to 180 degrees
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Connections:
- C1 pad 1: /VDRAIN -> VM
- C1 pad 2: Net-(U1-VCP) -> GND
- C10 pad 1: VM -> +5V_BUCK
- C11 pad 1: /BST -> +3V3
- C11 pad 2: /SW -> GND
- C12 pad 1: VBUCK -> /AMB_TMP
- C12 pad 2: /FB -> GND
- C13 pad 1: VBUCK -> /VGLS
- C14 pad 1: VBUCK -> /VCP
- C14 pad 2: Net-(C14-Pad2) -> /VDRAIN
- C15 pad 1: +3V3 -> /DVDD
- C17 pad 1: Net-(C17-Pad1) -> +5V_BUCK
- C17 pad 2: /MOTA -> GND
- C19 pad 1: /GHA -> +5V_BUCK
- C19 pad 2: /MOTA -> GND
- C2 pad 1: Net-(U1-VCC) -> VM
- C20 pad 1: /GLA -> VM
- C20 pad 2: /SPA -> GND
- C21 pad 1: /SPA -> /SPA_FILT
- C21 pad 2: /SNA -> /SNA_FILT
- C22 pad 1: /GHB -> /SW
- C22 pad 2: /MOTB -> /CB
- C23 pad 1: /GLB -> GND
- C23 pad 2: /SPB -> VM
- C24 pad 1: /SPB -> /SPB_FILT
- C24 pad 2: /SNB -> /SNB_FILT
- C25 pad 1: VM -> /SPC_FILT
- C25 pad 2: GND -> /SNC_FILT
- C27 pad 1: Net-(C27-Pad1) -> GND
- C27 pad 2: /MOTB -> VM
- C28 pad 1: /GHC -> GND
- C28 pad 2: /MOTC -> VM
- C29 pad 1: /GLC -> +3V3
- C29 pad 2: /SPC -> GND
- C3 pad 1: Net-(U1-VGLS) -> VM
- C30 pad 1: /SPC -> +3V3
- C30 pad 2: /SNC -> GND
- C31 pad 1: VM -> GND
- C31 pad 2: GND -> 5V_OR
- C33 pad 1: Net-(C33-Pad1) -> GND
- C33 pad 2: /MOTC -> +3V3
- C36 pad 1: VM -> 5V_OR
- C37 pad 1: VM -> +5V_BUCK
- C39 pad 1: /PHASE_TMP -> /QUAD_CH2
- C4 pad 1: Net-(U1-DVDD) -> VM
- C40 pad 1: /AMBIENT_TMP -> /QUAD_CH1
- C5 pad 1: +3V3 -> /PHASE_TMP
- C6 pad 1: Net-(U1-CPH) -> /CPL
- C6 pad 2: Net-(U1-CPL) -> /CPH
- C9 pad 1: VM -> GND
- C9 pad 2: GND -> VM
- CN1 pad 2: +3V3 -> GND
- CN1 pad 3: /ENC_CS -> /CANL
- CN1 pad 4: /SPI_SCK -> /CANH
- D1 pad 1: /SW -> Net-(D1-Pad1)
- D1 pad 2: GND -> /HEARBEAT
- J1 pad 1: Net-(J1-P) -> Net-(J1-Pin_1)
- J1 pad 2: GND -> /CANH
- L1 pad 2: VBUCK -> +5V_BUCK
- Q1 pad 4: /GHA -> /GHA_R
- Q2 pad 4: /GLA -> /GLA_R
- Q3 pad 4: /GHB -> /GHB_R
- Q4 pad 4: /GLB -> /GLB_R
- Q5 pad 4: /GHC -> /GHC_R
- Q6 pad 4: /GLC -> /GLC_R
- R1 pad 1: GND -> /SPA_FILT
- R1 pad 2: Net-(U1-RCL) -> /SPA
- R11 pad 1: VM -> /FB
- R11 pad 2: Net-(C27-Pad1) -> GND
- R14 pad 1: VM -> /CANL
- R14 pad 2: Net-(C33-Pad1) -> Net-(J1-Pin_1)
- R15 pad 1: Net-(U1-SOA) -> /IC
- R15 pad 2: /SOA -> /SOC
- R16 pad 1: Net-(U1-SOB) -> /IB
- R17 pad 1: /SPI_MISO -> +3V3
- R17 pad 2: +3V3 -> /PHASE_TMP
- R2 pad 1: VM -> /SNA_FILT
- R2 pad 2: Net-(U1-RT/SD) -> /SNA
- R21 pad 2: /PHASE_TMP -> /AMB_TMP
- R22 pad 2: /AMBIENT_TMP -> /FAULT
- R24 pad 1: +3V3 -> /BOOT0
- R24 pad 2: /ENC_CS -> GND
- R25 pad 1: +3V3 -> /GHC
- R25 pad 2: /FAULT -> /GHC_R
- R26 pad 1: Net-(D2-Pad1) -> /GHB
- R26 pad 2: GND -> /GHB_R
- R27 pad 1: Net-(D4-Pad1) -> /GHA
- R27 pad 2: /FAULT -> /GHA_R
- R28 pad 1: Net-(D6-Pad1) -> /GLC
- R28 pad 2: GND -> /GLC_R
- R3 pad 1: VBUCK -> Net-(D2-Pad1)
- R3 pad 2: /FB -> GND
- R4 pad 1: /FB -> Net-(D4-Pad1)
- R4 pad 2: GND -> /FAULT
- R5 pad 1: Net-(C14-Pad2) -> Net-(D6-Pad1)
- R6 pad 1: VM -> +5V_BUCK
- R6 pad 2: Net-(C17-Pad1) -> /FB
- TH2 pad 1: /AMBIENT_TMP -> /AMB_TMP
- U1 pad 1: GND -> /FB
- U1 pad 2: Net-(U1-VGLS) -> VM
- U1 pad 3: Net-(U1-CPL) -> VM
- U1 pad 4: Net-(U1-CPH) -> GND
- U1 pad 5: VM -> /SW
- U1 pad 6: /VDRAIN -> /CB
- U2 pad 1: GND -> unconnected-(U2-SSD-Pad1)
- U2 pad 2: +3V3 -> unconnected-(U2-A-Pad2)
- U2 pad 3: VBUCK -> unconnected-(U2-Z-Pad3)
- U2 pad 4: +3V3 -> /SPI_MOSI
- U4 pad 1: /MOTA -> /CPL
- U4 pad 2: /MOTB -> /CPH
- U4 pad 3: /MOTC -> VM
- U4 pad 4: GND -> /VDRAIN
- U4 pad 5: GND -> /VCP
- U7 pad 1: VM -> +3V3
- U7 pad 2: Net-(J1-P) -> unconnected-(U7-PC13-Pad2)
Routing:
- net /FAULT: track 69.2 -> 3.59 mm, vias 1 -> 0
- net Net-(U1-SOB): track 58.7 -> 0.00 mm, vias 2 -> 0
- net 5V_OR: track 0.00 -> 54.5 mm, vias 0 -> 2
- net Net-(U1-SOA): track 52.0 -> 0.00 mm, vias 2 -> 0
- net /GD_CS: track 64.9 -> 18.1 mm, vias 0 -> 2
- net /VSENA: track 0.00 -> 46.6 mm
- net /VSENB: track 0.00 -> 43.6 mm
- net VBUCK: track 41.6 -> 0.00 mm
- net /VSENC: track 0.00 -> 41.5 mm
- net /PHASE_TMP: track 80.1 -> 38.7 mm, vias 1 -> 0
- net /ENABLE: track 64.0 -> 23.1 mm, vias 1 -> 2
- net /ENC_CS: track 68.0 -> 27.4 mm, vias 0 -> 1
- net /USB_D+: track 0.00 -> 36.6 mm, vias 0 -> 2
- net /USB_D-: track 0.00 -> 35.7 mm, vias 0 -> 2
- net /MOTA: track 19.2 -> 54.2 mm, vias 19 -> 32
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- removed copper zone on F.Cu, net /FB
- removed copper zone on In1.Cu, net /MOTA
- removed copper zone on In1.Cu, net /MOTB
- removed copper zone on In1.Cu, net /MOTC
- removed copper zone on F.Cu, net /SPA
- removed copper zone on In1.Cu, net /SPA
- removed copper zone on In2.Cu, net /SPA
- removed copper zone on F.Cu, net /SPB
- removed copper zone on In1.Cu, net /SPB
- removed copper zone on In2.Cu, net /SPB
- removed copper zone on F.Cu, net /SPC
- removed copper zone on In1.Cu, net /SPC
- removed copper zone on In2.Cu, net /SPC
- removed copper zone on F.Cu, net /SW
- removed copper zone on B.Cu, net Net-(J1-P)
- removed copper zone on F.Cu, net Net-(J1-P)
- removed copper zone on In1.Cu, net Net-(J1-P)
- removed copper zone on In2.Cu, net Net-(J1-P)
- removed copper zone on F.Cu, net VBUCK
- removed copper zone on In1.Cu, net VM
Other:
- board size 117 x 75 mm -> 75 x 57 mm
- board text added: "3V3"
- board text added: "5V"
- board text added: "BOOT"
- board text added: "CAN"
- board text added: "GND"
- board text added: "MOTA"
- board text added: "MOTB"
- board text added: "MOTC"
- board text added: "QUAD ENC"
- board text added: "RESET"
- board text added: "SWD"
- board text added: "VM"
- board text removed: "Q1"
