File: bench_stm32_esc/bench_stm32_esc.kicad_sch (KiCad schematic)
At the start: 85 parts, among them J1 USB_C_Receptacle_USB2.0_16P, J2 XT60PW-M, Q1 CSD19532Q5B, Q2 CSD19532Q5B, SW1 SW_SPDT, U1 UCC27211ADRMR, U10 AS5047D, U11 USBLC6-2P6, U12 MR60PW-M.G.B, U4 AP2112K-3.3, U5 INA240A2D, U6 STM32G474RETx, U8 LM5164DDA, U9 TPD1E05U06DYA, X1 X322516MLB4SI

Commit message: Almost done rev 1.1
Parts:
- removed C1, C4: 10pF, PCM_JLCPCB:C_0603, symbol PCM_JLCPCB-Capacitors:0603,10pF
- removed C10: 1uF, PCM_JLCPCB:C_0805, symbol PCM_JLCPCB-Capacitors:0805,1uF
- removed C11, C12, C7, C8: 2.2nF, PCM_JLCPCB:C_0603, symbol PCM_JLCPCB-Capacitors:0603,2.2uF
- removed C13, C15, C16, C17, C18, C19, C20, C21, C23, C28, C3, C45, C46, C5: 100nF, PCM_JLCPCB:C_0603, symbol PCM_JLCPCB-Capacitors:0603,100nF
- removed C14: 10uF, PCM_JLCPCB:C_0603, symbol PCM_JLCPCB-Capacitors:0603,10uF
- removed C2, C25: 2.2uF, PCM_JLCPCB:C_0603, symbol PCM_JLCPCB-Capacitors:0603,2.2uF
- removed C22, C26, C6, C9: 1uF, PCM_JLCPCB:C_0603, symbol PCM_JLCPCB-Capacitors:0603,1uF
- removed C27: 47nF, PCM_JLCPCB:C_0603, symbol PCM_JLCPCB-Capacitors:0603,47nF
- removed C29, C32: VEJ331M2ATR-1816, footprints:VEJ331M2ATR-1816, symbol VEJ331M2ATR-1816:VEJ331M2ATR-1816
- removed C31, C36: 2.2nF, PCM_JLCPCB:C_0603, symbol PCM_JLCPCB-Capacitors:0603,2.2nF
- removed C34: 58pF, PCM_JLCPCB:C_0603, symbol PCM_JLCPCB-Capacitors:0603,33pF
- removed C39, C41, C44: 22uF, PCM_JLCPCB:C_0603, symbol PCM_JLCPCB-Capacitors:0603,22uF
- removed L2: SM7850-680MT, footprints:SM7850-680MT, symbol SM7850-680MT:SM7850-680MT
- removed Q1, Q2: CSD19532Q5B, Package_TO_SOT_SMD:TDSON-8-1, symbol Transistor_FET:CSD19532Q5B
- removed R1, R3: 3.3Ω, PCM_JLCPCB:R_0603, symbol PCM_JLCPCB-Resistors:0603,4.7Ω
- removed R10: 100kΩ, PCM_JLCPCB:R_0603, symbol PCM_JLCPCB-Resistors:0603,100kΩ
- removed R11: 383kΩ, PCM_JLCPCB:R_0805, symbol PCM_JLCPCB-Resistors:0805,300kΩ
- removed R12: 9.76kΩ, PCM_JLCPCB:R_0805, symbol PCM_JLCPCB-Resistors:0805,300kΩ
- removed R13, R6: 10kΩ, PCM_JLCPCB:R_0603, symbol PCM_JLCPCB-Resistors:0603,10kΩ
- removed R15: 150kΩ, PCM_JLCPCB:R_0603, symbol PCM_JLCPCB-Resistors:0603,150kΩ
- removed R16, R17: 5.1kΩ, PCM_JLCPCB:R_0603, symbol PCM_JLCPCB-Resistors:0603,5.1kΩ
- removed R19: 360kΩ, PCM_JLCPCB:R_0603, symbol PCM_JLCPCB-Resistors:0603,360kΩ
- removed R21: 470kΩ, PCM_JLCPCB:R_0603, symbol PCM_JLCPCB-Resistors:0603,470kΩ
- removed R22, R23: 330Ω, PCM_JLCPCB:R_0603, symbol PCM_JLCPCB-Resistors:0603,330Ω
- removed R24, R25: 4.7kΩ, PCM_JLCPCB:R_0603, symbol PCM_JLCPCB-Resistors:0603,4.7kΩ
- removed R4, R5: 2.7Ω, PCM_JLCPCB:R_0805, symbol PCM_JLCPCB-Resistors:0805,2.2Ω
- removed R8: 330kΩ, PCM_JLCPCB:R_0603, symbol PCM_JLCPCB-Resistors:0603,330kΩ
- removed SW1: SW_SPDT, symbol Switch:SW_SPDT
- removed TP1: TestPoint, TestPoint:TestPoint_Pad_1.5x1.5mm, symbol Connector:TestPoint
- removed U1: UCC27211ADRMR, easyeda2kicad:VSON-8_L4.0-W4.0-P0.80-TL-EP, symbol easyeda2kicad:UCC27211ADRMR
- removed U11: USBLC6-2P6, Package_TO_SOT_SMD:SOT-666, symbol Power_Protection:USBLC6-2P6
- removed U12: MR60PW-M.G.B, footprints:CONN-TH_MR60PW, symbol easyeda2kicad:MR60PW-M.G.B
- removed U5: INA240A2D, Package_SO:SOIC-8_3.9x4.9mm_P1.27mm, symbol Amplifier_Current:INA240A2D
- removed U8: LM5164DDA, Package_SO:HSOP-8-1EP_3.9x4.9mm_P1.27mm_EP2.41x3.1mm_ThermalVias, symbol Regulator_Switching:LM5164DDA
- removed U9: TPD1E05U06DYA, PCM_JLCPCB:D_SOD-523, symbol Power_Protection:TPD1E05U06DYA
- removed X1: X322516MLB4SI, PCM_JLCPCB:OSC-SMD_4P-L3.2-W2.5-BL, symbol PCM_JLCPCB-Crystals:Crystal, 16MHz, 9pF
- added C1, C25, C30, C31, C33, C4: 47pF, PCM_JLCPCB:C_0402, symbol PCM_JLCPCB-Capacitors:0402,47pF
- added C10, C11, C41, C43, C44, C56, C57, C58, C8: 220nF, PCM_JLCPCB:C_0805, symbol PCM_JLCPCB-Capacitors:0805,220nF
- added C100, C107, C15, C16, C17, C18, C2, C21, C22, C26, C27, C28, C3, C32, C34, C35, C38, C40, C45, C46, C5, C50, C52, C53, C54, C62, C63, C7, C76, C83, C86, C9, C97, C98, C99: 100nF, PCM_JLCPCB:C_0402, symbol PCM_JLCPCB-Capacitors:0402,100nF
- added C101, C102, C103, C104, C108, C109, C110, C111, C112, C113, C114, C51, C66, C67, C69, C70, C73: 1nF, PCM_JLCPCB:C_0402, symbol PCM_JLCPCB-Capacitors:0402,1nF
- added C105, C106, C77, C78, C79, C80, C82: FS55X226K101LRG, easyeda2kicad:C2220, symbol easyeda2kicad:FS55X226K101LRG
- added C12, C19, C24, C47, C48, C49, C59, C60, C61: 1uF, PCM_JLCPCB:C_0805, symbol PCM_JLCPCB-Capacitors:0805,1uF
- added C13, C20, C23, C29, C36, C39, C6, C93: 1uF, PCM_JLCPCB:C_0402, symbol PCM_JLCPCB-Capacitors:0402,1uF
- added C14: 4.7uF, PCM_JLCPCB:C_0402, symbol PCM_JLCPCB-Capacitors:0402,4.7uF
- added C55, C74, C96: 10uF, PCM_JLCPCB:C_0402, symbol PCM_JLCPCB-Capacitors:0603,10uF,(2)
- added C64, C65, C71, C75: 33nF, PCM_JLCPCB:C_0603, symbol PCM_JLCPCB-Capacitors:0603,33nF
- added C68, C72, C84, C95: 1.5nF, PCM_JLCPCB:C_0603, symbol PCM_JLCPCB-Capacitors:0603,1.5nF
- added C85, C87: 18pF, PCM_JLCPCB:C_0402, symbol PCM_JLCPCB-Capacitors:0402,18pF
- added C88, C92: 100nF, PCM_JLCPCB:C_0603, symbol PCM_JLCPCB-Capacitors:0603,100nF
- added C89: 18pF, PCM_JLCPCB:C_0603, symbol PCM_JLCPCB-Capacitors:0603,18pF
- added C90, C91: 15uF, PCM_JLCPCB:C_0603, symbol PCM_JLCPCB-Capacitors:0603,10uF
- added C94: 4.7uF, PCM_JLCPCB:C_1206, symbol PCM_JLCPCB-Capacitors:1206,4.7uF
- added D4: Red, PCM_JLCPCB:D_0805, symbol PCM_JLCPCB-Diodes:LED,0805,Red
- added D5: White, PCM_JLCPCB:D_0805, symbol PCM_JLCPCB-Diodes:LED,0805,White
- added FB4, FB5, FB6, FB7, FB8: (no value), PCM_JLCPCB:R_0402, symbol PCM_JLCPCB-Inductors:Ferrite,0603,(2)
- added H4: MountingHole, MountingHole:MountingHole_3.2mm_M3, symbol Mechanical:MountingHole
- added J3: Conn_ARM_SWD_TagConnect_TC2030-NL, Connector:Tag-Connect_TC2030-IDC-NL_2x03_P1.27mm_Vertical, symbol Connector:Conn_ARM_SWD_TagConnect_TC2030-NL
- added J4: Conn_01x02_Pin, Connector_PinHeader_2.54mm:PinHeader_1x02_P2.54mm_Vertical, symbol Connector:Conn_01x02_Pin
- added L1: MWSA1004S-220MT, easyeda2kicad:IND-SMD_L11.5-W10.0_FXL1040, symbol easyeda2kicad:MWSA1004S-220MT
- added NT1, NT2: NetTie_2, symbol Device:NetTie_2
- added NT3: NetTie_2, NetTie:NetTie-2_SMD_Pad0.5mm, symbol Device:NetTie_2
- added R1, R43, R44, R45, R46, R50, R52, R6, R8: 10kΩ, PCM_JLCPCB:R_0402, symbol PCM_JLCPCB-Resistors:0402,10kΩ
- added R10, R13, R22: 220Ω, PCM_JLCPCB:R_0402, symbol PCM_JLCPCB-Resistors:0402,220Ω
- added R11: 40.2kΩ, PCM_JLCPCB:R_0603, symbol PCM_JLCPCB-Resistors:0603,40.2kΩ
- added R12, R25, R3: 20kΩ, PCM_JLCPCB:R_0402, symbol PCM_JLCPCB-Resistors:0402,20kΩ
- added R14, R4, R5, R59, R60, R61, R62, R63, R64, R65, R66, R67, R68, R69, R70, R72, R75, R76, R77, R9: 20Ω, PCM_JLCPCB:C_0402, symbol PCM_JLCPCB-Resistors:0603,20Ω
- added R15, R16: 5.1kΩ, PCM_JLCPCB:R_0402, symbol PCM_JLCPCB-Resistors:0402,5.1kΩ
- added R17, R51: 100kΩ, PCM_JLCPCB:R_0402, symbol PCM_JLCPCB-Resistors:0402,100kΩ
- added R18, R2, R7: 1kΩ, PCM_JLCPCB:R_0402, symbol PCM_JLCPCB-Resistors:0402,1kΩ
- added R19, R20: 0Ω, PCM_JLCPCB:R_0603, symbol PCM_JLCPCB-Resistors:0603,0Ω
- added R21, R30, R34, R39: 1mΩ 3W, easyeda2kicad:R2512, symbol easyeda2kicad:LR2512-23R001F4
- added R23, R47: 120Ω, PCM_JLCPCB:R_0402, symbol PCM_JLCPCB-Resistors:0402,120Ω
- added R24, R42, R71: 3Ω, PCM_JLCPCB:R_0402, symbol PCM_JLCPCB-Resistors:0603,2.2Ω
- added R26, R28, R31, R37: 100kΩ, PCM_JLCPCB:R_0603, symbol PCM_JLCPCB-Resistors:0603,100kΩ
- added R27, R29, R32, R38: 4.22kΩ, PCM_JLCPCB:R_0603, symbol PCM_JLCPCB-Resistors:0603,7.5kΩ
- added R35, R36: 4.7kΩ, PCM_JLCPCB:R_0402, symbol PCM_JLCPCB-Resistors:0402,4.7kΩ
- added R48: 10kΩ, PCM_JLCPCB:R_0603, symbol PCM_JLCPCB-Resistors:0603,10kΩ
- added R49: 42.2kΩ, PCM_JLCPCB:R_0603, symbol PCM_JLCPCB-Resistors:0603,40.2kΩ
- added R53, R54, R55, R56, R57, R58, R73, R74: 10Ω, PCM_JLCPCB:R_0402, symbol PCM_JLCPCB-Resistors:0402,10Ω
- added S1, S2: Tactile Button, 160gf, PCM_JLCPCB:SW_TS-1088-AR02016, symbol PCM_JLCPCB-Connectors_Buttons:Tactile Button, 160gf, 12V, 50mA, 4.0mm
- added U1, U13, U8: LMG2100R044RARR, easyeda2kicad:QFN-17_L5.5-W4.5-P0.50-TL_LMG2100R044, symbol easyeda2kicad:LMG2100R044RARR
- added U11, U21, U22: TLV7041DBV, Package_TO_SOT_SMD:SOT-23-5, symbol Comparator:TLV7041DBV
- added U12: LMR38010FDDAR, easyeda2kicad:ESOP-8_L4.9-W3.9-P1.27-LS6.0-BL-EP3.1, symbol easyeda2kicad:LMR38010FDDAR
- added U14, U15, U16, U17: INA241A3xDDF, Package_TO_SOT_SMD:SOT-23-8, symbol Amplifier_Current:INA241A3xDDF
- added U18: REF3333AIDBZR, easyeda2kicad:SOT-23-3_L2.9-W1.6-P1.90-LS2.8-BR, symbol easyeda2kicad:REF3333AIDBZR
- added U19: XY130-9.5-3P, easyeda2kicad:CONN-TH_XY130-9.5-3P, symbol easyeda2kicad:XY130-9.5-3P
- added U2: LM66200DRLR, easyeda2kicad:SOT-583-8_L2.1-W1.2-P0.50-LS1.6-BL, symbol easyeda2kicad:LM66200DRLR
- added U20: USBLC6-2P6, Package_TO_SOT_SMD:SOT-666, symbol Power_Protection:USBLC6-2P6
- added U3: TCAN1044VDRBRQ1, easyeda2kicad:VSON-8_L3.0-W3.0-P0.65-BR-EP, symbol easyeda2kicad:TCAN1044VDRBRQ1
- added U5: TPD2E2U06DCK, Package_TO_SOT_SMD:SOT-323_SC-70, symbol Power_Protection:TPD2E2U06DCK
- added U7: S3B-PH-K-S-, easyeda2kicad:CONN-TH_3P-P2.00_S3B-PH-K-S-LF-SN, symbol easyeda2kicad:S3B-PH-K-S-
- added X1: X322524MOB4SI, easyeda2kicad:CRYSTAL-SMD_4P-L3.2-W2.5-BL, symbol easyeda2kicad:X322524MOB4SI
- J2: footprint footprints:AMASS_XT60PW-M -> easyeda2kicad:AMASS_XT60PW-M
Connections:
- net CSB is gone; now on net SPI_MOSI: U6.21 (PA7)
- net +3V3: now also C107.1, C14.1, C15.1, C16.1, C17.1, C18.1, C20.1, C21.1, C45.1, C54.1, C6.1, C63.1, C86.1, C9.1, C93.1, FB4.1, FB5.1, FB7.1, FB8.1, J3.1 (VCC), NT1.1, R1.1, R17.1, R18.1, R2.1, R35.1, R36.1, R7.1, R8.1, S2.1 (A), U11.5 (V+), U21.5 (V+), U22.5 (V+), U3.5 (NC/VIO)
- net +3V3A: now also U6.28 (VREF+), C22.1, C23.1, C83.1
- net +5V_USB: now also C39.1, U2.3 (VIN1); no longer U4.1 (VIN), U4.3 (EN)
- net AMB_TMP: now also C103.1, C26.1, R36.2, R63.2; no longer U6.14 (PA2)
- net BOOT0: now also R6.1, S2.2 (B)
- net CAN_RX: now also U6.58 (PB5), U3.4 (RXD); no longer U6.56 (PB3)
- net CAN_TX: now also U6.59 (PB6), U3.1 (TXD); no longer U6.50 (PA14), U6.57 (PB4)
- net GND: now also C1.2, C101.2, C102.2, C103.2, C104.2, C107.2, C108.2, C109.1, C110.1, C111.2, C112.1, C113.2, C114.2, C13.2, C14.2, C15.2, C16.2, C17.2, C18.2, C2.1, C20.2, C21.2, C22.2, C23.2, C25.2, C26.2, C27.2, C28.2, C29.2, C3.2, C30.2, C31.2, C32.2, C33.2, C34.2, C35.2, C36.2, C38.2, C39.2, C4.2, C40.2, C45.2, C46.1, C5.2, C50.2, C51.2, C54.2, C55.2, C6.2, C62.2, C63.2, C64.1, C65.1, C66.2, C67.2, C69.2, C7.2, C70.2, C71.1, C73.2, C74.2, C75.1, C76.2, C83.2, C85.2, C86.2, C87.2, C9.2, C90.2, C91.2, C92.2, C93.2, C94.2, C96.2, J3.5 (GND), R10.2, R12.2, R13.2, R15.2, R16.2, R19.2, R20.2, R22.2, R23.2, R25.2, R27.2, R29.2, R3.2, R32.2, R38.2, R43.2, R44.2, R45.2, R46.2, R48.1, R49.1, R50.2, R51.2, R52.2, R6.2, S1.1 (A), U1.15 (AGND), U11.2 (V-), U12.1 (GND), U12.9 (EP), U13.15 (AGND), U14.2 (GND), U14.3 (REF2), U14.4 (GND), U15.2 (GND), U15.3 (REF2), U15.4 (GND), U16.2 (GND), U16.3 (REF2), U16.4 (GND), U17.2 (GND), U17.3 (REF2), U17.4 (GND), U18.3 (GND), U2.1 (GND), U2.5 (GND), U20.2 (GND), U21.2 (V-), U22.2 (V-), U3.2 (GND), U3.8 (STB), U3.9 (EP), U5.3, U7.3, U8.15 (AGND), X1.2 (GND), X1.4 (GND); no longer J2.2 (N), J2.SH1 (SHIELD), J2.SH2 (SHIELD)
- net HSE_IN: now also C87.1, X1.3 (OSC2)
- net HSE_OUT: now also C85.1, X1.1 (OSC1)
- net NRST: now also C76.1, J3.3 (~{RESET}), S1.2 (B)
- net PHASE_TMP: now also C104.1, C28.1, R35.2, R64.2; no longer U6.13 (PA1)
- net SPI_MISO: now also U10.3 (MISO), U6.20 (PA6); no longer U6.53 (PC11)
- net SPI_MOSI: now also U10.4 (MOSI); no longer U6.52 (PC10)
- net SPI_SCK: now also U10.2 (CLK), U6.19 (PA5); no longer U6.54 (PC12)
- net SWCLK: now also U6.50 (PA14), J3.4 (SWCLK); no longer U6.49 (PA13)
- net USB_D+: now also U20.3 (I/O2)
- net USB_D-: now also U20.4 (I/O1)
- net USB_VBUS: now also U20.5 (VBUS)
- net VM: now also C10.1, C105.2, C106.2, C11.1, C12.1, C19.1, C24.1, C41.1, C43.1, C44.1, C47.1, C48.1, C49.1, C56.1, C57.1, C58.1, C59.1, C60.1, C61.1, C77.2, C78.2, C79.2, C8.1, C80.2, R28.1, R39.1, R74.1, U1.7 (VIN), U13.7 (VIN), U8.7 (VIN); no longer J2.1 (P)
- net VSENVM: now also C102.1, C65.2, R28.2, R29.1, R62.2; no longer U6.12 (PA0)
- net ENC_CS: now reaches U10.1 (~{CS})
- net ENC_CS: now also U6.13 (PA1), R8.2
- net at D2.1: now also R22.1
- net AMB_TMP_ADC: now reaches U6.10 (PC2)
- net AMB_TMP_ADC: now also R63.1
- net PHASE_TMP_ADC: now reaches U6.11 (PC3)
- net PHASE_TMP_ADC: now also R64.1
- net IB_ADC: now reaches U6.25 (PB1)
- net IB_ADC: now also R66.2
- net IA_ADC: now reaches U6.26 (PB2)
- net IA_ADC: now also R67.2
- net at U6.33 (PB11): now also R77.2
- net INLC: now reaches U6.38 (PC6)
- net INLC: now also R14.2, R45.1
- net INHC: now reaches U6.39 (PC7)
- net INHC: now also R46.1, R9.2
- net INLB: now reaches U6.40 (PC8)
- net INLB: now also R5.2, R50.1
- net INHB: now reaches U6.41 (PC9)
- net INHB: now also R4.2, R52.1
- net IDC_ADC: now reaches U6.8 (PC0)
- net IDC_ADC: now also R61.1
- net VDC_ADC: now reaches U6.9 (PC1)
- net VDC_ADC: now also R62.1
- net at U10.12 (VDD3V3): now also NT1.2
- net at D1.1: now also R13.1
- net CC2: now reaches J1.B5 (CC2)
- net CC2: now also R16.1
- net D-: now reaches J1.A7 (D-), J1.B7 (D-)
- net D-: now also U20.6 (I/O1)
- net D+: now reaches J1.A6 (D+), J1.B6 (D+)
- net D+: now also U20.1 (I/O2)
- net CC1: now reaches J1.A5 (CC1)
- net CC1: now also R15.1
- net CSA: no longer names the net of U6.17 (PA3)
- net CSC renamed IC_ADC
- net IC_ADC: now also R65.2
- net PWM_HA renamed INLA
- net INLA: now also R44.1, R60.2
- net PWM_HB renamed INHA
- net INHA: now also R43.1, R59.2
- net PWM_HC: no longer names the net of U6.44 (PA10)
- net PWM_LA renamed VC_ADC
- net VC_ADC: now also R68.2
- net PWM_LB renamed VB_ADC
- net VB_ADC: now also R69.2
- net PWM_LC renamed VA_ADC
- net VA_ADC: now also R70.2
- new net: C84.1, R73.2, U17.1 (-)
- new net: C46.2, FB7.2, U17.6 (V+)
- new net: C84.2, R74.2, U17.8 (+)
- new net: C40.1, FB8.2, U14.6 (V+)
- new net: C68.2, R54.2, U15.8 (+)
- new net: C112.2, R18.2, R25.1, U22.4 (-)
- new net: C97.1, R42.1
- new net: C68.1, R53.2, U15.1 (-)
- new net: C110.2, R12.1, R7.2, U21.4 (-)
- new net: C34.1, FB4.2, U15.6 (V+)
- new net: C2.2, FB5.2, U16.6 (V+)
- new net: C95.2, R56.2, U14.8 (+)
- new net: C109.2, R2.2, R3.1, U11.4 (-)
- new net: C52.1, R71.1
- new net: C113.1, R76.1, U22.3 (+)
- new net: NT2.1, U18.2 (OUT)
- new net: C72.2, R58.2, U16.8 (+)
- new net: C95.1, R55.2, U14.1 (-)
- new net: D4.1, R10.1
- new net: C111.1, R75.1, U21.3 (+)
- new net: C108.1, R72.1, U11.3 (+)
- new net: C72.1, R57.2, U16.1 (-)
- new net: C99.1, R24.1
- new net: D5.1, R23.1
- new net 5V_OR: C13.1, C62.1, FB6.1, U2.2 (VOUT), U2.7 (VOUT), U3.3 (VCC), U4.1 (VIN), U4.3 (EN)
- new net BOOT: C88.1, U12.7 (BOOT)
- new net CANH: J4.1 (Pin_1), U3.7 (CANH), U5.1, U7.1
- new net CANL: R47.2, U3.6 (CANL), U5.2, U7.2
- new net CANL_R: J4.2 (Pin_2), R47.1
- new net CSA+: R21.1, R56.1, U1.5 (SW)
- new net CSA-: R21.2, R26.1, R55.1, U19.3
- new net CSB+: R30.1, R54.1, U8.5 (SW)
- new net CSB-: R30.2, R31.1, R53.1, U19.2
- new net CSC+: R34.1, R58.1, U13.5 (SW)
- new net CSC-: R34.2, R37.1, R57.1
- new net FAULT: D4.2, U6.54 (PC12)
- new net FB: C89.1, R11.1, R48.2, U12.5 (FB)
- new net HBA: C100.1, R24.2, U1.10 (HB)
- new net HBB: C98.1, R42.2, U8.10 (HB)
- new net HBC: C53.1, R71.2, U13.10 (HB)
- new net HEARBEAT: U6.53 (PC11)
- new net HEARTBEAT: D5.2
- new net HIA: C25.1, R59.1, U1.12 (HI)
- new net HIB: C1.1, R4.1, U8.12 (HI)
- new net HIC: C31.1, R9.1, U13.12 (HI)
- new net HSA: C100.2, C99.2, U1.11 (HS)
- new net HSB: C97.2, C98.2, U8.11 (HS)
- new net HSC: C52.2, C53.2, U13.11 (HS)
- new net HW_OCP: C114.1, NT3.2, R77.1
- new net IA: C69.1, R67.1, R72.2, U14.5
- new net IB: C70.1, R66.1, R75.2, U15.5
- new net IC: C73.1, R65.1, R76.2, U16.5
- new net IDC: C101.1, R61.2, U17.5
- new net LIA: C30.1, R60.1, U1.13 (LI)
- new net LIB: C4.1, R5.1, U8.13 (LI)
- new net LIC: C33.1, R14.1, U13.13 (LI)
- new net OCP: NT3.1, R1.2, U11.1, U21.1, U22.1
- new net ON: R51.1, U2.4 (~{ON})
- new net PGND: C10.2, C105.1, C106.1, C11.2, C12.2, C19.2, C24.2, C41.2, C43.2, C44.2, C47.2, C48.2, C49.2, C56.2, C57.2, C58.2, C59.2, C60.2, C61.2, C77.1, C78.1, C79.1, C8.2, C80.1, C82.1, J2.2 (N), J2.SH1 (SHIELD), J2.SH2 (SHIELD), R19.1, R20.1, U1.17 (PGND), U1.6 (PGND), U13.17 (PGND), U13.6 (PGND), U8.17 (PGND), U8.6 (PGND)
- new net REFIN: C29.1, FB6.2, U18.1 (IN)
- new net RT: R49.2, U12.4 (RT/SYNC)
- new net ST: R17.2, U2.8 (ST)
- new net SW: C88.2, L1.1, U12.8 (SW)
- new net SWDIO: J3.2 (SWDIO), U6.49 (PA13)
- new net SWO: J3.6 (SWO), U6.56 (PB3)
- new net VBUCK: C35.1, C36.1, C5.1, C50.1, C55.1, C74.1, C89.2, C90.1, C91.1, C96.1, L1.2, R11.2, U1.14 (VCC), U13.14 (VCC), U2.6 (VIN2), U8.14 (VCC)
- new net VDC: C82.2, C92.1, C94.1, J2.1 (P), R39.2, R73.1, U12.2 (EN), U12.3 (VIN)
- new net VREF: C27.1, C3.1, C32.1, C38.1, C7.1, NT2.2, U14.7 (REF1), U15.7 (REF1), U16.7 (REF1), U17.7 (REF1)
- new net VSENA: C51.1, C64.2, R26.2, R27.1, R70.1
- new net VSENB: C66.1, C71.2, R31.2, R32.1, R69.1
- new net VSENC: C67.1, C75.2, R37.2, R38.1, R68.1
- no-connect marks 38 -> 48
Other:
- note added: "12-60V to 5.3V Buck"
- note added: "BUS Measurement"
- note added: "Input Voltage, Sensing, & Caps"
- note added: "OCP OR"
- note added: "Phase A Sensing"
- note added: "Phase B"
- note added: "Phase B Sensing"
- note added: "Phase C"
- note added: "Phase C Sensing"
- note added: "Reference Voltage"
- note added: "SPI AS5047D Encoder"
- note added: "SWD Connector"
- note added: "Star Connection"
- note removed: "12V Buck*"
- note removed: "Input Voltage"
- note removed: "SPI AS5047P Encoder"
- moved on the sheet: C37, C42, D1, D2, FB1, FB2, H1, H2, H3, J1, J2, TH1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
