File: bench_stm32_esc/bench_stm32_esc.kicad_sch (KiCad schematic)
At the start: 107 parts, among them CN1 S6B-PH-K-S-, CN10 Conn_02x19_Odd_Even, CN7 Conn_02x19_Odd_Even, J1 XT60PW-M, Q1 CSD19532Q5B, Q2 CSD19532Q5B, Q3 CSD19532Q5B, Q4 CSD19532Q5B, Q5 CSD19532Q5B, Q6 CSD19532Q5B, U1 DRV8353RSRGZT, U2 AMS1117, U3 TPD1E05U06DYA, U4 MR60PW-M.G.B, U7 TB60

Commit message: Revision 1.1
Parts:
- removed C1, C2, C3, C4: 1uF, PCM_JLCPCB:C_0603, symbol PCM_JLCPCB-Capacitors:0603,1uF
- removed C10, C25, C31, C7: 1uF, PCM_JLCPCB:C_0805, symbol PCM_JLCPCB-Capacitors:0805,1uF
- removed C12: 3.3nF, PCM_JLCPCB:C_0603, symbol PCM_JLCPCB-Capacitors:0603,3.3nF
- removed C13: 10uF, PCM_JLCPCB:C_CASE-A-3216-18(mm), symbol PCM_JLCPCB-Capacitors:CASE-A-3216-18(mm),10uF
- removed C14: 2.2uF, PCM_JLCPCB:C_0603, symbol PCM_JLCPCB-Capacitors:0603,2.2uF
- removed C15: 22uF, PCM_JLCPCB:C_CASE-A-3216-18(mm), symbol PCM_JLCPCB-Capacitors:CASE-A-3216-18(mm),10uF
- removed C16: VT10UF100V167RV0127, footprints:VT10UF100V167RV0127, symbol VT10UF100V167RV0127:VT10UF100V167RV0127
- removed C17, C19, C20, C22, C23, C27, C28, C29, C33, C34, C35: 2.2nF, PCM_JLCPCB:C_0603, symbol PCM_JLCPCB-Capacitors:0603,2.2uF
- removed C30: 1nF, PCM_JLCPCB:C_0603, symbol PCM_JLCPCB-Capacitors:0603,1nF
- removed C36, C37: VEJ331M2ATR-1816, footprints:VEJ331M2ATR-1816, symbol VEJ331M2ATR-1816:VEJ331M2ATR-1816
- removed C39, C40, C5, C9: 100nF, PCM_JLCPCB:C_0603, symbol PCM_JLCPCB-Capacitors:0603,100nF
- removed CN1: S6B-PH-K-S-, footprints:S6B-PH-K-S(LF)(SN), symbol S6B-PH-K-S(LF)(SN):S6B-PH-K-S-
- removed CN10, CN7: Conn_02x19_Odd_Even, Connector_PinSocket_2.54mm:PinSocket_2x19_P2.54mm_Vertical, symbol Connector_Generic:Conn_02x19_Odd_Even
- removed D1: DSK120, PCM_JLCPCB:D_SOD-123FL, symbol PCM_JLCPCB-Diodes:Schottky,DSK120
- removed J1: XT60PW-M, footprints:AMASS_XT60PW-M, symbol XT60PW-M:XT60PW-M
- removed L1: SMDRH104R-331MT, footprints:SMDRH104R-331MT, symbol SMDRH104R-331MT:SMDRH104R-331MT
- removed R1: 100kΩ, PCM_JLCPCB:R_0603, symbol PCM_JLCPCB-Resistors:0603,100kΩ
- removed R11, R14, R6: 2.7Ω, PCM_JLCPCB:R_0805, symbol PCM_JLCPCB-Resistors:0805,2.2Ω
- removed R15, R16: 56Ω, PCM_JLCPCB:R_0603, symbol PCM_JLCPCB-Resistors:0603,56Ω
- removed R17: 1kΩ, PCM_JLCPCB:R_0603, symbol PCM_JLCPCB-Resistors:0603,1kΩ
- removed R2: 274kΩ, PCM_JLCPCB:R_0603, symbol PCM_JLCPCB-Resistors:0603,100kΩ
- removed R21, R22: 4.7kΩ, PCM_JLCPCB:R_0603, symbol PCM_JLCPCB-Resistors:0603,4.7kΩ
- removed R24, R25, R3, R4: 10kΩ, PCM_JLCPCB:R_0603, symbol PCM_JLCPCB-Resistors:0603,10kΩ
- removed R26, R27, R28: 330Ω, PCM_JLCPCB:R_0603, symbol PCM_JLCPCB-Resistors:0603,330Ω
- removed R5: 2.2Ω, PCM_JLCPCB:R_0603, symbol PCM_JLCPCB-Resistors:0603,2.2Ω
- removed TP2, TP3, TP4, TP5: TestPoint, TestPoint:TestPoint_Pad_1.5x1.5mm, symbol Connector:TestPoint
- removed U1: DRV8353RSRGZT, footprints:QFN50P700X700X100-49N, symbol DRV8353RSRGZT:DRV8353RSRGZT
- removed U2: AMS1117, PCM_JLCPCB:SOT-223-3_L6.5-W3.4-P2.30-LS7.0-BR, symbol PCM_JLCPCB-Power:LDO, 3.3V, 1A
- removed U4: MR60PW-M.G.B, footprints:CONN-TH_MR60PW, symbol easyeda2kicad:MR60PW-M.G.B
- removed U7: TB60, footprints:TB60, symbol TB60:TB60
- added C1, C2, C3, C4, C7: EEHZC1K470V, easyeda2kicad:CAP-SMD_BD10.0-L10.3-W10.3-FD, symbol easyeda2kicad:EEHZC1K470V
- added C10, C17, C19: 47uF, PCM_JLCPCB:C_1206, symbol PCM_JLCPCB-Capacitors:0805,47uF
- added C12, C30, C31, C33, C41, C46, C47, C48, C49, C5, C50, C53, C64, C65, C76, C83: 100nF, PCM_JLCPCB:C_0402, symbol PCM_JLCPCB-Capacitors:0402,100nF
- added C13, C14, C15, C29, C36, C37, C42, C43, C45, C52, C93: 1uF, PCM_JLCPCB:C_0402, symbol PCM_JLCPCB-Capacitors:0402,1uF
- added C20, C22: 100nF, PCM_JLCPCB:C_0402, symbol PCM_JLCPCB-Capacitors:0603,100nF
- added C23, C27, C28: 1uF, PCM_JLCPCB:C_1206, symbol PCM_JLCPCB-Capacitors:1206,1uF
- added C25: 1nF, PCM_JLCPCB:C_0402, symbol PCM_JLCPCB-Capacitors:0603,1nF
- added C39, C40: 2.2nF, PCM_JLCPCB:C_0402, symbol PCM_JLCPCB-Capacitors:0402,2.2nF
- added C44: 4.7uF, PCM_JLCPCB:C_0402, symbol PCM_JLCPCB-Capacitors:0402,4.7uF
- added C51, C66, C67: 1nF, PCM_JLCPCB:C_0402, symbol PCM_JLCPCB-Capacitors:0402,1nF
- added C54, C55: 2.2uF, PCM_JLCPCB:C_0402, symbol PCM_JLCPCB-Capacitors:0603,2.2uF
- added C56, C57, C58: 10nF, PCM_JLCPCB:C_0402, symbol PCM_JLCPCB-Capacitors:0402,10nF
- added C61, C62, C63: 47nF, PCM_JLCPCB:C_0402, symbol PCM_JLCPCB-Capacitors:0603,47nF
- added C68, C69, C70, C71, C72, C73: 4.7uF, PCM_JLCPCB:C_1206, symbol PCM_JLCPCB-Capacitors:1206,4.7uF
- added C85, C87: 18pF, PCM_JLCPCB:C_0402, symbol PCM_JLCPCB-Capacitors:0402,18pF
- added C9: GRM32EC72A106KE05L, easyeda2kicad:C1210, symbol easyeda2kicad:GRM32EC72A106KE05L
- added CN1, CN2, CN3: 1053141104, easyeda2kicad:CONN-TH_4P-P2.50_MOLEX_1053141104, symbol easyeda2kicad:1053141104
- added D1: White, PCM_JLCPCB:D_0603, symbol PCM_JLCPCB-Diodes:LED,0603,White
- added D3: PESD2CAN,215, easyeda2kicad:SOT-23-3_L2.9-W1.3-P1.90-LS2.4-BR, symbol easyeda2kicad:PESD2CAN,215
- added FB1: (no value), PCM_JLCPCB:FB_0603, symbol PCM_JLCPCB-Inductors:Ferrite,0603
- added FB2: (no value), PCM_JLCPCB:FB_0603, symbol PCM_JLCPCB-Inductors:Ferrite,0603,(2)
- added J1: Conn_02x01, Connector_PinHeader_2.54mm:PinHeader_2x01_P2.54mm_Vertical, symbol Connector_Generic:Conn_02x01
- added J2: USB_C_Receptacle_USB2.0_16P, Connector_USB:USB_C_Receptacle_HRO_TYPE-C-31-M-12, symbol Connector:USB_C_Receptacle_USB2.0_16P
- added J3: Conn_ARM_SWD_TagConnect_TC2030-NL, Connector:Tag-Connect_TC2030-IDC-NL_2x03_P1.27mm_Vertical, symbol Connector:Conn_ARM_SWD_TagConnect_TC2030-NL
- added J4: Screw_Terminal_01x05, footprints:CUI_TB005_-762-05BE, symbol Connector:Screw_Terminal_01x05
- added L1: FNR4020S8R2MT, easyeda2kicad:IND-SMD_L4.0-W4.0_FNR40XXS, symbol easyeda2kicad:FNR4020S8R2MT
- added R1, R2, R42, R44, R45, R46, R47, R48, R49, R56: 100Ω, PCM_JLCPCB:R_0402, symbol PCM_JLCPCB-Resistors:0402,100Ω
- added R11: 19.1kΩ, PCM_JLCPCB:R_0402, symbol PCM_JLCPCB-Resistors:0402,100kΩ
- added R14: 120Ω, PCM_JLCPCB:R_0402, symbol PCM_JLCPCB-Resistors:0402,120Ω
- added R15, R16, R20: 56Ω, PCM_JLCPCB:R_0402, symbol PCM_JLCPCB-Resistors:0402,56kΩ
- added R17, R21: 4.7kΩ, PCM_JLCPCB:R_0402, symbol PCM_JLCPCB-Resistors:0402,4.7kΩ
- added R22, R24, R43, R50, R53: 10kΩ, PCM_JLCPCB:R_0402, symbol PCM_JLCPCB-Resistors:0402,10kΩ
- added R23, R51, R6: 100kΩ, PCM_JLCPCB:R_0402, symbol PCM_JLCPCB-Resistors:0402,100kΩ
- added R25, R26, R27, R28, R31, R32: 10Ω, PCM_JLCPCB:R_0402, symbol PCM_JLCPCB-Resistors:0402,10Ω
- added R29, R30: 5.1kΩ, PCM_JLCPCB:R_0402, symbol PCM_JLCPCB-Resistors:0402,5.1kΩ
- added R3, R4, R5: 330Ω, PCM_JLCPCB:R_0402, symbol PCM_JLCPCB-Resistors:0402,330Ω
- added R33, R35, R37: 383kΩ, PCM_JLCPCB:R_0402, symbol PCM_JLCPCB-Resistors:0805,300kΩ
- added R34, R36, R41, R55: 1kΩ, PCM_JLCPCB:R_0402, symbol PCM_JLCPCB-Resistors:0402,1kΩ
- added R38, R39, R40: 9.76kΩ, PCM_JLCPCB:R_0402, symbol PCM_JLCPCB-Resistors:0805,300kΩ
- added R52, R54: 20kΩ, PCM_JLCPCB:R_0402, symbol PCM_JLCPCB-Resistors:0402,20kΩ
- added S1, S2: Tactile Button, 160gf, PCM_JLCPCB:SW_TS-1088-AR02016, symbol PCM_JLCPCB-Connectors_Buttons:Tactile Button, 160gf, 12V, 50mA, 4.0mm
- added TP10, TP11, TP12, TP13, TP9: TestPoint, TestPoint:TestPoint_Pad_1.5x1.5mm, symbol Connector:TestPoint
- added U1: LMR51635YDDCR, easyeda2kicad:SOT-23-6_L2.9-W1.6-P0.95-LS2.8-BL, symbol easyeda2kicad:LMR51635YDDCR
- added U2: MA730, Package_DFN_QFN:QFN-16-1EP_3x3mm_P0.5mm_EP1.75x1.75mm, symbol Sensor_Magnetic:MA730
- added U20: USBLC6-2P6, Package_TO_SOT_SMD:SOT-666, symbol Power_Protection:USBLC6-2P6
- added U4: DRV8353SRTAR, easyeda2kicad:WQFN-40_L6.0-W6.0-P0.50-TL-EP4.5, symbol easyeda2kicad:DRV8353SRTAR
- added U5: LM66200DRLR, easyeda2kicad:SOT-583-8_L2.1-W1.2-P0.50-LS1.6-BL, symbol easyeda2kicad:LM66200DRLR
- added U6: AP2112K-3.3, Package_TO_SOT_SMD:SOT-23-5, symbol Regulator_Linear:AP2112K-3.3
- added U7: STM32G474RETx, Package_QFP:LQFP-64_10x10mm_P0.5mm, symbol MCU_ST_STM32G4:STM32G474RETx
- added U8: TCAN1462VDRBRQ1, easyeda2kicad:DFN-8_L3.0-W3.0-P0.65-TL-EP2.4, symbol easyeda2kicad:TCAN1462VDRBRQ1
- added X1: X322524MOB4SI, easyeda2kicad:CRYSTAL-SMD_4P-L3.2-W2.5-BL, symbol easyeda2kicad:X322524MOB4SI
- C11: value 10nF -> 100nF; footprint PCM_JLCPCB:C_0603 -> PCM_JLCPCB:C_0402; LCSC C43253 -> C162178; Manufacturer (none) -> Murata Electronics; Part (none) -> GRM155R62A104KE14D; Temperature Coefficient X7R -> X5R
- C18, C26, C32: footprint PCM_JLCPCB:C_0603 -> PCM_JLCPCB:C_0402; Capacitance 2.2uF -> 2.2nF; LCSC C113804 -> C576731; Part CC0603KRX7R0BB222 -> CC0402KRX7R0BB222; Temperature Coefficient X5R -> X7R
- C21, C24: footprint PCM_JLCPCB:C_0603 -> PCM_JLCPCB:C_0402; LCSC C43847 -> C527013; Manufacturer FH (Guangdong Fenghua Advanced Tech) -> YAGEO; Part 0603B102K101NT -> CC0402KRX7R0BB102
- C8: footprint PCM_JLCPCB:C_0603 -> PCM_JLCPCB:C_0402; LCSC C15725 -> C162178; Manufacturer Samsung Electro-Mechanics -> Murata Electronics; Part CL10B104KC8NNNC -> GRM155R62A104KE14D; Temperature Coefficient X7R -> X5R
- Q1, Q2, Q3, Q4, Q5, Q6: value CSD19532Q5B -> IAUCN08S7N019ATMA1; LCSC C2832190 -> C33993693
- R12, R8, R9: value 7mΩ -> 2mΩ; LCSC C393073 -> C2994640; Manafacturer TA-I Tech -> Milliohm; Part No RLP25FEGMR007 -> HoLLR2512-3W-2mR-1%
Connections:
- net BST is gone; now on net +3V3: C11.1
- net +3V3: now also C29.1, C30.1, C33.2, C44.1, C45.1, C46.1, C47.1, C48.1, C49.1, C53.1, C93.1, FB1.2, J3.1 (VCC), R17.1, R21.1, R22.1, R23.1, R43.1, R55.1, S2.1 (A), TP13.1, U2.13 (VDD), U4.24 (VREF), U6.5 (VOUT), U7.1 (VBAT), U7.16 (VDD), U7.32 (VDD), U7.48 (VDD), U7.64 (VDD), U8.5 (NC/VIO)
- net ENABLE: now also U4.31 (ENABLE), U7.57 (PB4)
- net ENC_CS: now also U2.5 (~{CS}), U7.33 (PB11)
- net FAULT: now also R22.2, R4.2, U4.26 (nFAULT)
- net FB: now also R11.1, R6.2, U1.1 (FB)
- net GD_CS: now also R43.2, U4.30 (nSCS), U7.52 (PC10)
- net GHA: now also R27.1, U4.6 (GHA); no longer Q1.4 (G)
- net GHB: now also R26.1, U4.15 (GHB); no longer Q3.4 (G)
- net GHC: now also R25.1, U4.16 (GHC); no longer Q5.4 (G)
- net GLA: now also R32.1, U4.8 (GLA); no longer Q2.4 (G)
- net GLB: now also R31.1, U4.13 (GLB); no longer Q4.4 (G)
- net GLC: now also R28.1, U4.18 (GLC); no longer Q6.4 (G)
- net GND: now also C11.2, C1.2, C10.2, C12.2, C13.2, C15.2, C17.2, C19.2, C2.2, C20.2, C23.1, C27.1, C28.1, C29.2, C3.2, C30.2, C31.1, C33.1, C36.2, C37.2, C39.2, C4.2, C40.2, C41.2, C42.2, C43.2, C44.2, C45.2, C46.2, C47.2, C48.2, C49.2, C5.2, C50.2, C51.2, C52.2, C53.2, C54.2, C55.2, C56.2, C57.2, C58.2, C61.2, C62.2, C63.2, C64.2, C65.2, C66.2, C67.2, C68.2, C69.2, C7.2, C70.2, C71.2, C72.2, C73.2, C76.2, C83.2, C85.2, C87.2, C9.1, C93.2, CN1.1, CN1.2, CN2.1, CN2.2, CN3.1, D3.3, J2.A1 (GND), J2.A12 (GND), J2.B1 (GND), J2.B12 (GND), J2.SH (SHIELD), J3.5 (GND), J4.4 (Pin_4), R11.2, R24.2, R29.2, R3.2, R30.2, R38.2, R39.2, R40.2, R5.2, R51.2, R52.2, R54.2, R56.2, S1.1 (A), TP10.1, TP11.1, TP9.1, U1.4 (GND), U2.10 (TEST), U2.17 (PAD), U2.8 (GND), U20.2 (GND), U4.25 (AGND), U4.39 (GND), U4.41 (EP), U5.1 (GND), U5.5 (GND), U6.2 (GND), U7.15 (VSS), U7.27 (VSSA), U7.31 (VSS), U7.47 (VSS), U7.63 (VSS), U8.2 (GND), U8.8 (STB), U8.9 (EP), X1.2 (GND), X1.4 (GND)
- net INHA: now also U4.32 (INHA), U7.43 (PA9)
- net INHB: now also U4.34 (INHB), U7.41 (PC9)
- net INHC: now also U4.36 (INHC), U7.39 (PC7)
- net INLA: now also U4.33 (INLA), U7.42 (PA8)
- net INLB: now also U4.35 (INLB), U7.40 (PC8)
- net INLC: now also U4.37 (INLC), U7.38 (PC6)
- net MOTA: now also J4.2 (Pin_2), R33.1
- net MOTB: now also J4.3 (Pin_3), R35.1
- net MOTC: now also J4.5 (Pin_5), R37.1
- net PHASE_TMP: now also C5.1, R17.2, R49.1
- net SHA: now also U4.7 (SHA)
- net SHB: now also U4.14 (SHB)
- net SHC: now also U4.17 (SHC)
- net SNA: now also R2.2; no longer C21.2
- net SNB: now also R44.2; no longer C24.2
- net SNC: now also R46.2
- net SOA: now also R20.2, U4.23 (SOA)
- net SOB: now also R16.2, U4.22 (SOB)
- net SPA: now also R1.2; no longer C21.1
- net SPB: now also R42.2; no longer C24.1
- net SPC: now also R45.2
- net SPI_MISO: now also R55.2, U2.7 (MISO), U4.27 (SDO), U7.20 (PA6)
- net SPI_MOSI: now also U2.4 (MOSI), U4.28 (SDI), U7.21 (PA7)
- net SPI_SCK: now also U2.12 (SCLK), U4.29 (SCLK), U7.19 (PA5)
- net SW: now also C22.1, L1.1, U1.5 (SW); no longer C11.2
- net VDRAIN: now also C14.2, U4.4 (VDRAIN)
- net VM: now also C1.1, C2.1, C20.1, C23.2, C27.2, C28.2, C3.1, C4.1, C68.1, C69.1, C7.1, C70.1, C71.1, C72.1, C73.1, C9.2, J4.1 (Pin_1), U1.2 (EN), U1.3 (VIN), U4.3 (VM)
- net VSENVM: now also R47.1
- net CPH: now reaches C6.2
- net CPH: now also U4.2 (CPH)
- net CPL: now reaches C6.1
- net CPL: now also U4.1 (CPL)
- net at D6.1: now also R5.1
- net at D2.1: now also R3.1
- net at D4.1: now also R4.1
- net AMBIENT_TMP renamed AMB_TMP
- net AMB_TMP: now also C12.1, R21.2, R48.1
- new net: J1.1 (Pin_1), R14.2
- new net: D1.1, R56.1
- new net +3V3A: C50.1, C52.1, C83.1, FB1.1, U7.28 (VREF+), U7.29 (VDDA)
- new net +5V_BUCK: C10.1, C17.1, C19.1, C37.1, L1.2, R6.1, U5.6 (VIN2)
- new net +5V_USB: C42.1, C55.1, FB2.2, U5.3 (VIN1)
- new net 5V_OR: C31.2, C36.1, C43.1, CN3.2, TP12.1, U5.2 (VOUT), U5.7 (VOUT), U6.1 (VIN), U6.3 (EN), U8.3 (VCC)
- new net AMB_TMP_ADC: C64.1, R48.2, U7.10 (PC2)
- new net BOOT0: R24.1, S2.2 (B), U7.61 (PB8)
- new net CANH: CN1.4, CN2.4, D3.1, J1.2 (Pin_2), U8.7 (CANH)
- new net CANL: CN1.3, CN2.3, D3.2, R14.1, U8.6 (CANL)
- new net CAN_RX: U7.58 (PB5), U8.4 (RXD)
- new net CAN_TX: U7.59 (PB6), U8.1 (TXD)
- new net CB: C22.2, U1.6 (CB)
- new net CC1: J2.A5 (CC1), R30.1
- new net CC2: J2.B5 (CC2), R29.1
- new net D+: J2.A6 (D+), J2.B6 (D+), U20.1 (I/O2)
- new net D-: J2.A7 (D-), J2.B7 (D-), U20.6 (I/O1)
- new net DVDD: C15.1, U4.38 (DVDD)
- new net GHA_R: Q1.4 (G), R27.2
- new net GHB_R: Q3.4 (G), R26.2
- new net GHC_R: Q5.4 (G), R25.2
- new net GLA_R: Q2.4 (G), R32.2
- new net GLB_R: Q4.4 (G), R31.2
- new net GLC_R: Q6.4 (G), R28.2
- new net HEARBEAT: D1.2, U7.18 (PA4)
- new net HSE_IN: C87.1, U7.5 (PF0), X1.3 (OSC2)
- new net HSE_OUT: C85.1, U7.6 (PF1), X1.1 (OSC1)
- new net IA: C56.1, R20.1, U7.37 (PB15)
- new net IB: C57.1, R16.1, U7.36 (PB14)
- new net IC: C58.1, R15.1, U7.35 (PB13)
- new net NRST: C76.1, J3.3 (~{RESET}), S1.2 (B), U7.7 (PG10)
- new net ON: R51.1, U5.4 (~{ON})
- new net PHASE_TMP_ADC: C65.1, R49.2, U7.11 (PC3)
- new net QUAD_CH1: C40.1, R50.2, R52.1, U7.12 (PA0)
- new net QUAD_CH1_CONN: CN3.4, R50.1
- new net QUAD_CH2: C39.1, R53.2, R54.1, U7.13 (PA1)
- new net QUAD_CH2_CONN: CN3.3, R53.1
- new net SNA_FILT: C21.2, R2.1, U4.10 (SNA)
- new net SNB_FILT: C24.2, R44.1, U4.11 (SNB)
- new net SNC_FILT: C25.2, R46.1, U4.20 (SNC)
- new net SOC: R15.2, U4.21 (SOC)
- new net SPA_FILT: C21.1, R1.1, U4.9 (SPA)
- new net SPB_FILT: C24.1, R42.1, U4.12 (SPB)
- new net SPC_FILT: C25.1, R45.1, U4.19 (SPC)
- new net ST: R23.2, U5.8 (ST)
- new net SWCLK: J3.4 (SWCLK), U7.50 (PA14)
- new net SWDIO: J3.2 (SWDIO), U7.49 (PA13)
- new net SWO: J3.6 (SWO), U7.56 (PB3)
- new net USB_D+: U20.3 (I/O2), U7.46 (PA12)
- new net USB_D-: U20.4 (I/O1), U7.45 (PA11)
- new net USB_VBUS: C54.1, FB2.1, J2.A4 (VBUS), J2.A9 (VBUS), J2.B4 (VBUS), J2.B9 (VBUS), U20.5 (VBUS)
- new net VA_ADC: C51.1, R41.1, U7.26 (PB2)
- new net VB_ADC: C66.1, R36.1, U7.25 (PB1)
- new net VCP: C14.1, U4.5 (VCP)
- new net VC_ADC: C67.1, R34.1, U7.24 (PB0)
- new net VDC_ADC: C41.1, R47.2, U7.9 (PC1)
- new net VGLS: C13.1, U4.40 (VGLS)
- new net VSENA: C61.1, R33.2, R40.1, R41.2
- new net VSENB: C62.1, R35.2, R36.2, R39.1
- new net VSENC: C63.1, R34.2, R37.2, R38.1
- no-connect marks 51 -> 27
Other:
- note added: "CAN Transciever + Connectors"
- note added: "Crystal"
- note added: "Power ORing + LDO"
- note added: "Quadrature Encoder Connector"
- note added: "SPI MA730 Encoder"
- note added: "STM32G474"
- note added: "SWD Connector"
- note added: "USB-C Connector"
- note added: "VM to 5V Buck"
- note removed: "Buck + LDO"
- note removed: "CAN Transciever"
- note removed: "Phase Output"
- note removed: "SPI Encoder Connector"
- note removed: "STM32G4 Nucleo Connectors"
- moved on the sheet: C21, C6, C8, D2, D4, D6, H1, H2, H3, H4, NT1, NT2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
